File: Hardware/PCB/PCB_Mere/KiCad/PCB_Mere_V1.kicad_pcb (KiCad board)
At the start: 2 copper layers, 1 part, among them U1 STM32H723ZGTx

Commit message: Add files via upload
Parts:
- added CN1: FTSH-107-01-L-DV-K-A, EasyEDA:HDR-SMD_14P-P1.27_FTSH-107-01-L-DV-K-A, F.Cu at (118.0, 115.0)
- added CN2: BM08B-GHS-TBT, EasyEDA:CONN-SMD_BM08B-GHS-TBT-LF-SN, F.Cu at (53.8, 56.3)
- added CN3: BM08B-GHS-TBT, EasyEDA:CONN-SMD_BM08B-GHS-TBT-LF-SN, F.Cu at (53.8, 62.9)
- added CN4: BM08B-GHS-TBT, EasyEDA:CONN-SMD_BM08B-GHS-TBT-LF-SN, F.Cu at (53.8, 69.5)
- added CN5: B2B-PH-K-S_FILLE_ALIM, EasyEDA:CONN-TH_B2B-PH-K-S, F.Cu at (87.6, 56.9)
- added CN6: B2B-PH-K-S_GNSS_ALIM, EasyEDA:CONN-TH_B2B-PH-K-S, F.Cu at (87.6, 62.7)
- added H1: PZ254-1-20-Z-8.5, EasyEDA:HDR-TH_20P-P2.54-V-M, F.Cu at (169.2, 70.5)
- added H2: PZ254-1-20-Z-8.5, EasyEDA:HDR-TH_20P-P2.54-V-M, F.Cu at (169.7, 118.5)
- added TF1: 473092651, EasyEDA:TF-SMD_47309-2285, F.Cu at (218.5, 82.9)
- added U2: LORA1276-C1-868MHZ, EasyEDA:COMM-SMD_LORA1276-C1-915MHZ, F.Cu at (170.7, 38.8)
- added U3: ESP32C3-SUPERMINI, EasyEDA:COMM-SMD_16P-L22.5-W18.0-P2.54-TL, F.Cu at (210.5, 103.7)
- added U4: BNO055, EasyEDA:LGA-28_L5.2-W3.8-P0.50-BL, F.Cu at (128.6, 56.8)
- added U5: B8B-PH-K-S-, EasyEDA:CONN-TH_B8B-PH-K-S-LF-SN, F.Cu at (93.6, 45.4)
- added U6: B8B-PH-K-S_FILS, EasyEDA:CONN-TH_B8B-PH-K-S-LF-SN, F.Cu at (93.6, 51.2)
- U1: value STM32H723ZGTx -> STM32H723ZGT6; footprint Package_QFP:LQFP-144_20x20mm_P0.5mm -> EasyEDA:LQFP-144_L20.0-W20.0-P0.50-LS22.0-BL
- moved U1 10.6 mm to (160.0, 93.8), turned to -45 degrees
Connections:
- U1 pad 106: unconnected-(U1-VCAP-Pad106) -> Net-(C3-Pad1)
- U1 pad 107: Net-(U1-VSS-Pad107) -> NRST
- U1 pad 108: unconnected-(U1-VDD-Pad108) -> NRST
- U1 pad 120: Net-(U1-VSS-Pad107) -> NRST
- U1 pad 121: unconnected-(U1-VDD-Pad121) -> NRST
- U1 pad 130: Net-(U1-VSS-Pad107) -> NRST
- U1 pad 131: unconnected-(U1-VDD-Pad131) -> NRST
- U1 pad 138: unconnected-(U1-BOOT0-Pad138) -> Net-(U1-BOOT0)
- U1 pad 143: unconnected-(U1-PDR_ON-Pad143) -> NRST
- U1 pad 144: unconnected-(U1-VDD-Pad144) -> NRST
- U1 pad 16: Net-(U1-VSS-Pad107) -> NRST
- U1 pad 17: unconnected-(U1-VDD-Pad17) -> NRST
- U1 pad 25: unconnected-(U1-NRST-Pad25) -> Net-(U1-NRST)
- U1 pad 30: unconnected-(U1-VDD-Pad30) -> NRST
- U1 pad 31: unconnected-(U1-VSSA-Pad31) -> NRST
- U1 pad 32: unconnected-(U1-VREF+-Pad32) -> NRST
- U1 pad 33: unconnected-(U1-VDDA-Pad33) -> NRST
- U1 pad 38: Net-(U1-VSS-Pad107) -> NRST
- U1 pad 39: unconnected-(U1-VDD-Pad39) -> NRST
- U1 pad 51: Net-(U1-VSS-Pad107) -> NRST
- U1 pad 52: unconnected-(U1-VDD-Pad52) -> NRST
- U1 pad 6: unconnected-(U1-VBAT-Pad6) -> NRST
- U1 pad 61: Net-(U1-VSS-Pad107) -> NRST
- U1 pad 62: unconnected-(U1-VDD-Pad62) -> NRST
- U1 pad 71: unconnected-(U1-VCAP-Pad71) -> Net-(C2-Pad2)
- U1 pad 72: unconnected-(U1-VDD-Pad72) -> NRST
- U1 pad 83: Net-(U1-VSS-Pad107) -> NRST
- U1 pad 84: unconnected-(U1-VDD-Pad84) -> NRST
- U1 pad 94: Net-(U1-VSS-Pad107) -> NRST
- U1 pad 95: unconnected-(U1-VDD33USB-Pad95) -> NRST

Commit message: push du kicad
Parts:
- removed CN3, CN4: BM08B-GHS-TBT, EasyEDA:CONN-SMD_BM08B-GHS-TBT-LF-SN
- removed CN5: B2B-PH-K-S_FILLE_ALIM, EasyEDA:CONN-TH_B2B-PH-K-S
- removed CN6: B2B-PH-K-S_GNSS_ALIM, EasyEDA:CONN-TH_B2B-PH-K-S
- removed H2: PZ254-1-20-Z-8.5, EasyEDA:HDR-TH_20P-P2.54-V-M
- added H3: PZ254-1-10-Z-8.5_EL, EasyEDA:HDR-TH_10P-P2.54-V-M, F.Cu at (182.9, 122.5)
- added SW1: NRST_BTN, EasyEDA:KEY-SMD_4P-L3.5-W2.9-P1.48-LS4.3-TL, F.Cu at (203.0, 97.6)
- added SW2: BOOT_BTN, EasyEDA:KEY-SMD_4P-L3.5-W2.9-P1.48-LS4.3-TL, F.Cu at (203.0, 101.5)
- added U7: B10B-PH-K-S-_SCRN/JOY/ALIM, EasyEDA:CONN-TH_B10B-PH-K-S-LF-SN, F.Cu at (139.0, 110.7)
- CN2: value BM08B-GHS-TBT -> B4B-PH-K-S_GNSS; footprint EasyEDA:CONN-SMD_BM08B-GHS-TBT-LF-SN -> EasyEDA:CONN-TH_B4B-PH-K-S
- H1: value PZ254-1-20-Z-8.5 -> PZ254-1-20-Z-8.5_AZ
- U5: value B8B-PH-K-S- -> B8B-PH-K-S-_TACTIL
- moved CN2 150.4 mm to (203.0, 74.9), turned to 120 degrees
- moved U5 100.6 mm to (154.3, 125.6), turned to -27 degrees
- moved U4 58.0 mm to (153.2, 109.2)
- moved U6 51.1 mm to (137.4, 77.6), turned to -115 degrees
- moved U2 44.5 mm to (155.0, 80.5), turned to -135 degrees
- moved CN1 27.5 mm to (135.5, 93.7), turned to -90 degrees
- moved TF1 22.2 mm to (238.5, 92.6)
- moved U1 16.3 mm to (176.2, 95.0)
- moved U3 14.7 mm to (220.7, 93.1)
- moved H1 6.13 mm to (170.4, 64.5)
Connections:
- net Net-(U4-nBOOT_LOAD_PIN) renamed IMU-BOOT
- net Net-(U4-nRESET) renamed IMU-RST
- CN1 pad 03: NRST -> +3.3V
- CN1 pad 05: NRST -> +3.3V
- CN1 pad 07: NRST -> +3.3V
- CN1 pad 11: NRST -> +3.3V
- CN1 pad 12: NRST -> NRST_STM
- CN2 pad 1: unconnected-(CN2-Pad1) -> +3.3V
- CN2 pad 2: unconnected-(CN2-Pad2) -> +3.3V
- CN2 pad 3: unconnected-(CN2-Pad3) -> GNSS_UART5_TX
- CN2 pad 4: unconnected-(CN2-Pad4) -> GNSS_UART5_RX
- H1 pad 1: unconnected-(H1-Pad1) -> +3.3V
- H1 pad 2: unconnected-(H1-Pad2) -> +3.3V
- TF1 pad 4: NRST -> +3.3V
- TF1 pad 6: NRST -> +3.3V
- TF1 pad G1: NRST -> +3.3V
- TF1 pad G2: NRST -> +3.3V
- TF1 pad G4: NRST -> +3.3V
- U1 pad 107: NRST -> +3.3V
- U1 pad 108: NRST -> +3.3V
- U1 pad 120: NRST -> +3.3V
- U1 pad 121: NRST -> +3.3V
- U1 pad 130: NRST -> +3.3V
- U1 pad 131: NRST -> +3.3V
- U1 pad 143: NRST -> +3.3V
- U1 pad 144: NRST -> +3.3V
- U1 pad 16: NRST -> +3.3V
- U1 pad 17: NRST -> +3.3V
- U1 pad 22: unconnected-(U1-PF10-Pad22) -> SCREEN_RST_GPIO_Output
- U1 pad 25: Net-(U1-NRST) -> NRST_STM
- U1 pad 30: NRST -> +3.3V
- U1 pad 31: NRST -> +3.3V
- U1 pad 32: NRST -> +3.3V
- U1 pad 33: NRST -> +3.3V
- U1 pad 38: NRST -> +3.3V
- U1 pad 39: NRST -> +3.3V
- U1 pad 40: unconnected-(U1-PA4-Pad40) -> TACTIL_SPI6_NSS
- U1 pad 41: unconnected-(U1-PA5-Pad41) -> TACTIL_SPI6_SCK
- U1 pad 42: unconnected-(U1-PA6-Pad42) -> TACTIL_SPI6_MISO
- U1 pad 43: unconnected-(U1-PA7-Pad43) -> TACTIL_SPI6_MOSI
- U1 pad 44: unconnected-(U1-PC4-Pad44) -> TACTIL_GPIO_EXTI4
- U1 pad 45: unconnected-(U1-PC5-Pad45) -> ETAT-B-ON/OFF_GPIO_Input
- U1 pad 46: unconnected-(U1-PB0-Pad46) -> BONUS1_GPIO
- U1 pad 47: unconnected-(U1-PB1-Pad47) -> BONUS2_GPIO
- U1 pad 51: NRST -> +3.3V
- U1 pad 52: NRST -> +3.3V
- U1 pad 6: NRST -> +3.3V
- U1 pad 61: NRST -> +3.3V
- U1 pad 62: NRST -> +3.3V
- U1 pad 72: NRST -> +3.3V
- U1 pad 83: NRST -> +3.3V
- U1 pad 84: NRST -> +3.3V
- U1 pad 94: NRST -> +3.3V
- U1 pad 95: NRST -> +3.3V
- U2 pad 1: NRST -> +3.3V
- U2 pad 10: NRST -> +3.3V
- U2 pad 13: Net-(U2-VCC) -> +3.3V
- U2 pad 8: NRST -> +3.3V
- U3 pad 1: ESP32_UART7_RX -> ESP32_UART7_TX
- U3 pad 14: Net-(U3-3V3) -> +3.3V
- U3 pad 15: NRST -> +3.3V
- U3 pad 16: Net-(U3-5V) -> +3.3V
- U3 pad 2: ESP32_UART7_TX -> ESP32_UART7_RX
- U4 pad 18: NRST -> +3.3V
- U4 pad 2: NRST -> +3.3V
- U4 pad 25: NRST -> +3.3V
- U4 pad 28: Net-(U4-VDDIO) -> unconnected-(U4-VDDIO-Pad28)
- U4 pad 3: NRST -> +3.3V
- U4 pad 5: NRST -> +3.3V
- U4 pad 6: NRST -> +3.3V
- U5 pad 1: NRST -> BONUS2_GPIO
- U5 pad 2: unconnected-(U5-Pad2) -> BONUS1_GPIO
- U5 pad 3: unconnected-(U5-Pad3) -> ETAT-B-ON/OFF_GPIO_Input
- U5 pad 4: unconnected-(U5-Pad4) -> TACTIL_GPIO_EXTI4
- U5 pad 5: unconnected-(U5-Pad5) -> TACTIL_SPI6_MOSI
- U5 pad 6: unconnected-(U5-Pad6) -> TACTIL_SPI6_MISO
- U5 pad 7: unconnected-(U5-Pad7) -> TACTIL_SPI6_SCK
- U5 pad 8: unconnected-(U5-Pad8) -> TACTIL_SPI6_NSS
- U6 pad 1: NRST -> +3.3V
- U6 pad 2: Net-(C31-Pad2) -> +3.3V
- U6 pad 3: Net-(C32-Pad2) -> +3.3V
- U6 pad 7: LIDAR_UART8_RX -> LIDAR_UART8_TX
- U6 pad 8: LIDAR_UART8_TX -> LIDAR_UART8_RX

Commit message: Dernière version Schématique
Parts:
- added C1: 100n, Capacitor_SMD:C_0201_0603Metric, F.Cu at (83.8, 70.8)
- added C10: 100n, Capacitor_SMD:C_0201_0603Metric, F.Cu at (83.8, 77.8)
- added C11: 100n, Capacitor_SMD:C_0201_0603Metric, F.Cu at (83.8, 79.5)
- added C12: 100n, Capacitor_SMD:C_0201_0603Metric, F.Cu at (86.3, 70.8)
- added C13: 100n, Capacitor_SMD:C_0201_0603Metric, F.Cu at (86.3, 72.5)
- added C14: 100n, Capacitor_SMD:C_0201_0603Metric, F.Cu at (86.3, 74.3)
- added C15: 100n, Capacitor_SMD:C_0201_0603Metric, F.Cu at (86.3, 76.0)
- added C16: 100n, Capacitor_SMD:C_0201_0603Metric, F.Cu at (86.3, 77.8)
- added C17: 100n, Capacitor_SMD:C_0201_0603Metric, F.Cu at (86.3, 79.5)
- added C18: 100n, Capacitor_SMD:C_0201_0603Metric, F.Cu at (88.7, 70.8)
- added C19: 100n, Capacitor_SMD:C_0201_0603Metric, F.Cu at (88.7, 72.5)
- added C2: 2,2µ, Capacitor_SMD:C_0201_0603Metric, F.Cu at (85.1, 51.6)
- added C20: 10µ, Capacitor_SMD:C_0201_0603Metric, F.Cu at (85.1, 60.3)
- added C21: 100n, Capacitor_SMD:C_0201_0603Metric, F.Cu at (88.7, 74.3)
- added C22: 1u, Capacitor_SMD:C_0201_0603Metric, F.Cu at (93.2, 81.5)
- added C23: 120n, Capacitor_SMD:C_0201_0603Metric, F.Cu at (93.2, 83.3)
- added C24: 100n, Capacitor_SMD:C_0201_0603Metric, F.Cu at (93.2, 85.0)
- added C25: 22p, Capacitor_SMD:C_0201_0603Metric, F.Cu at (95.6, 81.5)
- added C26: 22p, Capacitor_SMD:C_0201_0603Metric, F.Cu at (95.6, 83.3)
- added C27: 100n, Capacitor_SMD:C_0201_0603Metric, F.Cu at (95.6, 85.0)
- added C28: 4,7u, Capacitor_SMD:C_0201_0603Metric, F.Cu at (89.6, 51.6)
- added C29: 10n, Capacitor_SMD:C_0402_1005Metric, F.Cu at (89.6, 53.3)
- added C3: 2,2µ, Capacitor_SMD:C_0201_0603Metric, F.Cu at (85.1, 53.3)
- added C30: 10n, Capacitor_SMD:C_0402_1005Metric, F.Cu at (85.1, 62.1)
- added C31: 100n, Capacitor_SMD:C_0201_0603Metric, F.Cu at (93.2, 70.8)
- added C32: 100n, Capacitor_SMD:C_0201_0603Metric, F.Cu at (93.2, 72.5)
- added C33: 100n, Capacitor_SMD:C_0201_0603Metric, F.Cu at (152.7, 96.7)
- added C34: 100n, Capacitor_SMD:C_0201_0603Metric, F.Cu at (146.7, 96.6)
- added C35: 100n, Capacitor_SMD:C_0201_0603Metric, F.Cu at (145.1, 96.6)
- added C36: 100n, Capacitor_SMD:C_0201_0603Metric, F.Cu at (93.2, 74.3)
- added C37: 100n, Capacitor_SMD:C_0201_0603Metric, F.Cu at (93.2, 76.0)
- added C38: 100n, Capacitor_SMD:C_0201_0603Metric, F.Cu at (93.2, 77.8)
- added C4: 1µ, Capacitor_SMD:C_0201_0603Metric, F.Cu at (85.1, 55.1)
- added C5: 1µ, Capacitor_SMD:C_0201_0603Metric, F.Cu at (85.1, 56.8)
- added C6: 100n, Capacitor_SMD:C_0201_0603Metric, F.Cu at (83.8, 72.5)
- added C7: 0,1µ, Capacitor_SMD:C_0201_0603Metric, F.Cu at (85.1, 58.6)
- added C8: 100n, Capacitor_SMD:C_0201_0603Metric, F.Cu at (83.8, 74.3)
- added C9: 100n, Capacitor_SMD:C_0201_0603Metric, F.Cu at (83.8, 76.0)
- added H2: MountingHole_Pad, footprint:MountingHole_3.2mm_M3, F.Cu at (170.5, 58.3)
- added H4: MountingHole_Pad, footprint:MountingHole_3.2mm_M3, F.Cu at (205.1, 93.9)
- added H5: MountingHole_Pad, footprint:MountingHole_3.2mm_M3, F.Cu at (155.0, 114.8)
- added R10: 47k, Resistor_SMD:R_0201_0603Metric, F.Cu at (94.5, 51.6)
- added R11: 47k, Resistor_SMD:R_0201_0603Metric, F.Cu at (94.5, 53.3)
- added R12: 10k, Resistor_SMD:R_0201_0603Metric, F.Cu at (94.5, 55.1)
- added R13: 10k, Resistor_SMD:R_0201_0603Metric, F.Cu at (103.6, 51.9)
- added R14: 10k, Resistor_SMD:R_0201_0603Metric, F.Cu at (85.1, 63.8)
- added R15: 330, Resistor_SMD:R_0201_0603Metric, F.Cu at (198.2, 114.5)
- added R16: 1k, Resistor_SMD:R_0201_0603Metric, F.Cu at (198.3, 115.5)
- added R2: 47k, Resistor_SMD:R_0201_0603Metric, F.Cu at (89.6, 55.1)
- added R3: 47k, Resistor_SMD:R_0201_0603Metric, F.Cu at (89.6, 56.8)
- added R4: 47k, Resistor_SMD:R_0201_0603Metric, F.Cu at (89.6, 58.6)
- added R5: 2,2k, Resistor_SMD:R_0201_0603Metric, F.Cu at (92.0, 51.6)
- added R6: 2,2k, Resistor_SMD:R_0201_0603Metric, F.Cu at (98.3, 72.6)
- added R6: 2,2k, Resistor_SMD:R_0201_0603Metric, F.Cu at (92.0, 53.3)
- added R7: 2,2k, Resistor_SMD:R_0201_0603Metric, F.Cu at (98.3, 74.3)
- added R7: 2,2k, Resistor_SMD:R_0201_0603Metric, F.Cu at (92.0, 55.1)
- added R8: 10k, Resistor_SMD:R_0201_0603Metric, F.Cu at (92.0, 56.8)
- added R9: 10k, Resistor_SMD:R_0201_0603Metric, F.Cu at (92.0, 58.6)
- added U8: A-SP1102AR6GHC-A01-2C, EasyEDA:LED-SMD_4P-L3.0-W1.5_A-SP1102AR6GHC-A01-2C, F.Cu at (200.2, 114.2)
- moved SW1 5.39 mm to (202.3, 102.9)
- moved SW2 5.39 mm to (202.3, 106.8)
- moved U4 4.22 mm to (152.8, 105.0)
Connections:
- U1 pad 80: LED2_DEBUG_GPIO_Output -> unconnected-(U1-PD11-Pad80)

Commit message: Nouvelles empreintes de mounting holes et plusieurs court circuits retirés du schematic
Parts:
- H2, H4, H5: footprint footprint:MountingHole_3.2mm_M3 -> MountingHole:MountingHole_3.2mm_M3_DIN965_Pad_TopBottom
- moved H4 2.64 mm to (204.0, 91.5)
Changed lines of the file:
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@@
 		)
 	)
-	(footprint "footprint:MountingHole_3.2mm_M3"
+	(footprint "MountingHole:MountingHole_3.2mm_M3_DIN965_Pad_TopBottom"
 		(layer "F.Cu")
 		(at 155 114.8)
-		(descr "Mounting Hole 3.2mm, M3, no annular, generated by kicad-footprint-generator mountinghole.py")
-		(tags "mountinghole M3")
+		(descr "Mounting Hole 3.2mm, M3, generated by kicad-footprint-generator mountinghole.py")
+		(tags "mountinghole M3 DIN965")
 		(property "Reference" "H5"
-			(at 0 -4.15 0)
+			(at 0 -3.75 0)
 			(layer "F.SilkS")
 			(effects
@@
 		)
 		(property "Value" "MountingHole_Pad"
-			(at 0 4.15 0)
+			(at 0 3.75 0)
 			(layer "F.Fab")
 			(effects
@@
 		(fp_circle
 			(center 0 0)
-			(end 3.2 0)
+			(end 2.8 0)
 			(stroke
 				(width 0.15)
@@
 		(fp_circle
 			(center 0 0)
-			(end 3.45 0)
+			(end 3.05 0)
 			(stroke
 				(width 0.05)
@@
 			)
 		)
-		(pad "" np_thru_hole circle
+		(pad "1" thru_hole circle
 			(at 0 0)
-			(size 3.2 3.2)
+			(size 3.6 3.6)
 			(drill 3.2)
 			(layers "*.Cu" "*.Mask")
+			(remove_unused_layers no)
+			(net "+3.3V")
+			(pinfunction "1_1")
+			(pintype "input")
+			(zone_connect 2)
+		)
+		(pad "1" connect circle
+			(at 0 0)
+			(size 5.6 5.6)
+			(layers "F.Cu" "F.Mask")
+			(net "+3.3V")
+			(pinfunction "1_1")
+			(pintype "input")
+			(zone_connect 2)
+		)
+		(pad "1" connect circle
+			(at 0 0)
+			(size 5.6 5.6)
+			(layers "B.Cu" "B.Mask")
+			(net "+3.3V")
+			(pinfunction "1_1")
+			(pintype "input")
+			(zone_connect 2)
 		)
 		(embedded_fonts no)
@@
 		)
 	)
-	(footprint "footprint:MountingHole_3.2mm_M3"
+	(footprint "MountingHole:MountingHole_3.2mm_M3_DIN965_Pad_TopBottom"
 		(layer "F.Cu")
-		(at 205.1 93.9)
-		(descr "Mounting Hole 3.2mm, M3, no annular, generated by kicad-footprint-generator mountinghole.py")
-		(tags "mountinghole M3")
+		(at 204 91.5)
+		(descr "Mounting Hole 3.2mm, M3, generated by kicad-footprint-generator mountinghole.py")
+		(tags "mountinghole M3 DIN965")
 		(property "Reference" "H4"
-			(at 0 -4.15 0)
+			(at 0 -3.75 0)
 			(layer "F.SilkS")
 			(effects
@@
 		)
 		(property "Value" "MountingHole_Pad"
-			(at 0 4.15 0)
+			(at 0 3.75 0)
 			(layer "F.Fab")
 			(effects
@@
 		(fp_circle
 			(center 0 0)
-			(end 3.2 0)
+			(end 2.8 0)
 			(stroke
 				(width 0.15)
@@
 		(fp_circle
 			(center 0 0)
-			(end 3.45 0)
+			(end 3.05 0)
 			(stroke
 				(width 0.05)
@@
 			)
 		)
-		(pad "" np_thru_hole circle
+		(pad "1" thru_hole circle
 			(at 0 0)
-			(size 3.2 3.2)
+			(size 3.6 3.6)
 			(drill 3.2)
 			(layers "*.Cu" "*.Mask")
+			(remove_unused_layers no)
+			(net "+3.3V")
+			(pinfunction "1_1")
+			(pintype "input")
+			(zone_connect 2)
+		)
+		(pad "1" connect circle
+			(at 0 0)
+			(size 5.6 5.6)
+			(layers "F.Cu" "F.Mask")
+			(net "+3.3V")
+			(pinfunction "1_1")
+			(pintype "input")
+			(zone_connect 2)
+		)
+		(pad "1" connect circle
+			(at 0 0)
+			(size 5.6 5.6)
+			(layers "B.Cu" "B.Mask")
+			(net "+3.3V")
+			(pinfunction "1_1")
+			(pintype "input")
+			(zone_connect 2)
 		)
 		(embedded_fonts no)
@@
 		)
 	)
-	(footprint "footprint:MountingHole_3.2mm_M3"
+	(footprint "MountingHole:MountingHole_3.2mm_M3_DIN965_Pad_TopBottom"
 		(layer "F.Cu")
 		(at 170.5 58.3)
-		(descr "Mounting Hole 3.2mm, M3, no annular, generated by kicad-footprint-generator mountinghole.py")
-		(tags "mountinghole M3")
+		(descr "Mounting Hole 3.2mm, M3, generated by kicad-footprint-generator mountinghole.py")
+		(tags "mountinghole M3 DIN965")
 		(property "Reference" "H2"
-			(at 0 -4.15 0)
+			(at 0 -3.75 0)
 			(layer "F.SilkS")
 			(effects
@@
 		)
 		(property "Value" "MountingHole_Pad"
-			(at 0 4.15 0)
+			(at 0 3.75 0)
 			(layer "F.Fab")
 			(effects
@@
 		(fp_circle
 			(center 0 0)
-			(end 3.2 0)
+			(end 2.8 0)
 			(stroke
 				(width 0.15)
@@
 		(fp_circle
 			(center 0 0)
-			(end 3.45 0)
+			(end 3.05 0)
 			(stroke
 				(width 0.05)
@@
 			)
 		)
-		(pad "" np_thru_hole circle
+		(pad "1" thru_hole circle
 			(at 0 0)
-			(size 3.2 3.2)
+			(size 3.6 3.6)
 			(drill 3.2)
 			(layers "*.Cu" "*.Mask")
+			(remove_unused_layers no)
+			(net "+3.3V")
+			(pinfunction "1_1")
+			(pintype "input")
+			(zone_connect 2)
+		)
+		(pad "1" connect circle
+			(at 0 0)
+			(size 5.6 5.6)
+			(layers "F.Cu" "F.Mask")
+			(net "+3.3V")
+			(pinfunction "1_1")
+			(pintype "input")
+			(zone_connect 2)
+		)
+		(pad "1" connect circle
+			(at 0 0)
+			(size 5.6 5.6)
+			(layers "B.Cu" "B.Mask")
+			(net "+3.3V")
+			(pinfunction "1_1")
+			(pintype "input")
+			(zone_connect 2)
 		)
 		(embedded_fonts no)

Commit message: avancement schematic fils
Connections:
- C1 pad 1: Net-(C1-Pad1) -> GND
- C10 pad 2: +3.3V -> GND
- C11 pad 2: +3.3V -> GND
- C12 pad 2: +3.3V -> GND
- C13 pad 2: +3.3V -> GND
- C14 pad 2: +3.3V -> GND
- C15 pad 2: +3.3V -> GND
- C16 pad 2: +3.3V -> GND
- C17 pad 2: +3.3V -> GND
- C18 pad 2: +3.3V -> GND
- C19 pad 2: +3.3V -> GND
- C2 pad 1: +3.3V -> GND
- C20 pad 2: +3.3V -> GND
- C21 pad 2: +3.3V -> GND
- C22 pad 1: +3.3V -> GND
- C23 pad 1: +3.3V -> GND
- C24 pad 1: +3.3V -> GND
- C25 pad 1: +3.3V -> GND
- C26 pad 1: +3.3V -> GND
- C27 pad 2: +3.3V -> GND
- C28 pad 1: +3.3V -> GND
- C29 pad 2: +3.3V -> GND
- C3 pad 2: +3.3V -> GND
- C30 pad 1: +3.3V -> GND
- C31 pad 2: +3.3V -> GND
- C32 pad 1: +3.3V -> +5V
- C32 pad 2: +3.3V -> GND
- C33 pad 2: +3.3V -> GND
- C34 pad 1: +3.3V -> GND
- C34 pad 2: +3.3V -> +5V
- C35 pad 2: +3.3V -> GND
- C36 pad 1: +3.3V -> GND
- C36 pad 2: +3.3V -> +5V
- C37 pad 1: +3.3V -> GND
- C38 pad 1: +3.3V -> GND
- C38 pad 2: +3.3V -> +5V
- C4 pad 1: Net-(C1-Pad1) -> GND
- C5 pad 1: Net-(C5-Pad1) -> +3.3V
- C5 pad 2: +3.3V -> GND
- C6 pad 1: Net-(C5-Pad1) -> +3.3V
- C6 pad 2: +3.3V -> GND
- C7 pad 2: +3.3V -> GND
- C8 pad 2: +3.3V -> GND
- C9 pad 2: +3.3V -> GND
- CN1 pad 05: +3.3V -> GND
- CN1 pad 07: +3.3V -> GND
- CN1 pad 11: +3.3V -> GND
- CN2 pad 1: +3.3V -> GND
- CN2 pad 2: +3.3V -> +5V
- H1 pad 1: +3.3V -> GND
- H1 pad 2: +3.3V -> +5V
- H2 pad 1: +3.3V -> GND
- H4 pad 1: +3.3V -> GND
- H5 pad 1: +3.3V -> GND
- R14 pad 2: +3.3V -> GND
- SW1 pad 2: +3.3V -> GND
- TF1 pad 6: +3.3V -> GND
- TF1 pad G1: +3.3V -> GND
- TF1 pad G2: +3.3V -> GND
- TF1 pad G4: +3.3V -> GND
- U1 pad 107: +3.3V -> GND
- U1 pad 120: +3.3V -> GND
- U1 pad 130: +3.3V -> GND
- U1 pad 16: +3.3V -> GND
- U1 pad 31: +3.3V -> GND
- U1 pad 38: +3.3V -> GND
- U1 pad 51: +3.3V -> GND
- U1 pad 61: +3.3V -> GND
- U1 pad 83: +3.3V -> GND
- U1 pad 94: +3.3V -> GND
- U2 pad 1: +3.3V -> GND
- U2 pad 10: +3.3V -> GND
- U2 pad 8: +3.3V -> GND
- U3 pad 15: +3.3V -> GND
- U3 pad 16: +3.3V -> +5V
- U4 pad 18: +3.3V -> GND
- U4 pad 2: +3.3V -> GND
- U4 pad 25: +3.3V -> GND
- U4 pad 5: +3.3V -> GND
- U4 pad 6: +3.3V -> GND
- U6 pad 1: +3.3V -> GND
- U6 pad 2: +3.3V -> +5V
- U7 pad 1: +3.3V -> GND
- U8 pad 3: +3.3V -> GND
- U8 pad 4: +3.3V -> GND
Other:
- copper layers 2 -> 4
