File: Hardware/PCB/PCB_Mere/KiCad/PCB_Mere_V1.kicad_pcb (KiCad board)
At the start: 4 copper layers, 113.4 x 80.1 mm, 79 parts, among them CN1 FTSH-107-01-L-DV-K-A, CN2 B4B-PH-K-S_GNSS, SW1 NRST_BTN, SW2 BOOT_BTN, U1 STM32H723ZGT6, U2 LORA1276-C1-868MHZ, U3 ESP32C3-SUPERMINI, U4 BNO055, U5 B8B-PH-K-S-_TACTIL, U6 B8B-PH-K-S_FILS, U7 B10B-PH-K-S-_SCRN/JOY/ALIM, U8 A-SP1102AR6GHC-A01-2C, X1 X322525MOB4SI, X2 X701532768KGD4GI

Commit message: last version
Parts:
- moved R7 0.07 mm to (154.5, 97.2)

Commit message: last version
Parts:
- added C42: 100n, Capacitor_SMD:C_0402_1005Metric, F.Cu at (156.5, 61.3)
- moved C39 2.61 mm to (154.0, 61.3)
Connections:
- H1 pad 3: +3.3V -> GND
- H1 pad 4: unconnected-(H1-Pad4) -> +3.3V
- H1 pad 5: unconnected-(H1-Pad5) -> +3.3V
- H1 pad 6: unconnected-(H1-Pad6) -> GND
- H1 pad 7: unconnected-(H1-Pad7) -> GND
- H1 pad 8: unconnected-(H1-Pad8) -> GND
Routing:
- net +3.3V: track 109.6 -> 112.6 mm
- net +5V: track 12.0 -> 14.0 mm, vias 2 -> 1
Other:
- outline, holes or cut-outs redrawn

Commit message: last version
Parts:
- removed C35: 100n, Capacitor_SMD:C_0402_1005Metric
- BOOT_BTN-2: renamed from SW2; value BOOT_BTN -> switch
- C7: value 0,1µ -> 100n
- NRST_BTN-1: renamed from SW1; value NRST_BTN -> switch
Routing:
- net +3.3V: track 112.6 -> 107.2 mm
Changed lines of the file:
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@@
 	(footprint "Capacitor_SMD:C_0402_1005Metric"
 		(layer "F.Cu")
-		(at 231.75 87.88 90)
-		(descr "Capacitor SMD 0402 (1005 Metric), square (rectangular) end terminal, IPC-7351 nominal, (Body size source: IPC-SM-782 page 76, https://www.pcb-3d.com/wordpress/wp-content/uploads/ipc-sm-782a_amendment_1_and_2.pdf)")
-		(tags "capacitor")
-		(property "Reference" "C35"
-			(at 0 -1.16 90)
-			(layer "F.SilkS")
-			(effects
-				(font
-					(size 1 1)
-					(thickness 0.15)
-				)
-			)
-		)
-		(property "Value" "100n"
-			(at 0 1.16 90)
-			(layer "F.Fab")
-			(effects
-				(font
-					(size 1 1)
-					(thickness 0.15)
-				)
-			)
-		)
-		(property "Datasheet" ""
-			(at 0 0 90)
-			(layer "F.Fab")
-			(hide yes)
-			(effects
-				(font
-					(size 1.27 1.27)
-				)
-			)
-		)
-		(property "Description" "Unpolarized capacitor, small symbol"
-			(at 0 0 90)
-			(layer "F.Fab")
-			(hide yes)
-			(effects
-				(font
-					(size 1.27 1.27)
-				)
-			)
-		)
-		(property "KiLib_Generator" "SMD_2terminal_chip_molded"
-			(at 0 0 90)
-			(layer "F.SilkS")
-			(hide yes)
-			(effects
-				(font
-					(size 1 1)
-					(thickness 0.15)
-				)
-			)
-		)
-		(property "LCSC Part" "C49062"
-			(at 0 0 90)
-			(unlocked yes)
-			(layer "F.Fab")
-			(hide yes)
-			(effects
-				(font
-					(size 1 1)
-					(thickness 0.15)
-				)
-			)
-		)
-		(property ki_fp_filters "C_*")
-		(sheetname "/Composant_Mère/")
-		(sheetfile "Composant_Mere.kicad_sch")
-		(units
-			(unit
-				(name "A")
-				(pins "1" "2")
-			)
-		)
-		(attr smd)
-		(duplicate_pad_numbers_are_jumpers no)
-		(fp_line
-			(start -0.107836 -0.36)
-			(end 0.107836 -0.36)
-			(stroke
-				(width 0.12)
-				(type solid)
-			)
-			(layer "F.SilkS")
-		)
-		(fp_line
-			(start -0.107836 0.36)
-			(end 0.107836 0.36)
-			(stroke
-				(width 0.12)
-				(type solid)
-			)
-			(layer "F.SilkS")
-		)
-		(fp_rect
-			(start -0.91 -0.46)
-			(end 0.91 0.46)
-			(stroke
-				(width 0.05)
-				(type solid)
-			)
-			(fill no)
-			(layer "F.CrtYd")
-		)
-		(fp_rect
-			(start -0.5 -0.25)
-			(end 0.5 0.25)
-			(stroke
-				(width 0.1)
-				(type solid)
-			)
-			(fill no)
-			(layer "F.Fab")
-		)
-		(fp_text user "${REFERENCE}"
-			(at 0 0 90)
-			(layer "F.Fab")
-			(effects
-				(font
-					(size 0.25 0.25)
-					(thickness 0.04)
-				)
-			)
-		)
-		(pad "1" smd roundrect
-			(at -0.48 0 90)
-			(size 0.56 0.62)
-			(layers "F.Cu" "F.Mask" "F.Paste")
-			(roundrect_rratio 0.25)
-			(net "+3.3V")
-			(pintype "passive")
-		)
-		(pad "2" smd roundrect
-			(at 0.48 0 90)
-			(size 0.56 0.62)
-			(layers "F.Cu" "F.Mask" "F.Paste")
-			(roundrect_rratio 0.25)
-			(net "GND")
-			(pintype "passive")
-		)
-		(embedded_fonts no)
-		(model "${KICAD10_3DMODEL_DIR}/Capacitor_SMD.3dshapes/C_0402_1005Metric.step"
-			(offset
-				(xyz 0 0 0)
-			)
-			(scale
-				(xyz 1 1 1)
-			)
-			(rotate
-				(xyz 0 0 0)
-			)
-		)
-	)
-	(footprint "Capacitor_SMD:C_0402_1005Metric"
-		(layer "F.Cu")
 		(at 176.1 78.2 45)
 		(descr "Capacitor SMD 0402 (1005 Metric), square (rectangular) end terminal, IPC-7351 nominal, (Body size source: IPC-SM-782 page 76, https://www.pcb-3d.com/wordpress/wp-content/uploads/ipc-sm-782a_amendment_1_and_2.pdf)")
@@
 		(layer "F.Cu")
 		(at 201.48 102.9 180)
-		(property "Reference" "SW1"
+		(property "Reference" "NRST_BTN-1"
 			(at -4.5 -0.1 0)
 			(layer "F.SilkS")
@@
 			)
 		)
-		(property "Value" "NRST_BTN"
+		(property "Value" "switch"
 			(at 0 4.74 0)
 			(layer "F.Fab")
@@
 			(size 1.05 1.15)
 			(layers "F.Cu" "F.Mask" "F.Paste")
-			(net "unconnected-(SW1-Pad1)")
+			(net "unconnected-(NRST_BTN-1-Pad1)")
 			(pinfunction "1_1")
 			(pintype "unspecified+no_connect")
@@
 			(size 1.05 1.15)
 			(layers "F.Cu" "F.Mask" "F.Paste")
-			(net "unconnected-(SW1-Pad2')")
+			(net "unconnected-(NRST_BTN-1-Pad2')")
 			(pinfunction "2'_2'")
 			(pintype "unspecified+no_connect")
@@
 			)
 		)
-		(property "Value" "0,1µ"
+		(property "Value" "100n"
 			(at 0 1.16 0)
 			(layer "F.Fab")
@@
 		(layer "F.Cu")
 		(at 201.5 107.3)
-		(property "Reference" "SW2"
+		(property "Reference" "BOOT_BTN-2"
 			(at 4.7 -0.8 0)
 			(layer "F.SilkS")
@@
 			)
 		)
-		(property "Value" "BOOT_BTN"
+		(property "Value" "switch"
 			(at 0 4.74 0)
 			(layer "F.Fab")
@@
 			(size 1.05 1.15)
 			(layers "F.Cu" "F.Mask" "F.Paste")
-			(net "unconnected-(SW2-Pad1')")
+			(net "unconnected-(BOOT_BTN-2-Pad1')")
 			(pinfunction "1'_1'")
 			(pintype "unspecified+no_connect")
@@
 			(size 1.05 1.15)
 			(layers "F.Cu" "F.Mask" "F.Paste")
-			(net "unconnected-(SW2-Pad2)")
+			(net "unconnected-(BOOT_BTN-2-Pad2)")
 			(pinfunction "2_2")
 			(pintype "unspecified+no_connect")
@@
 	)
 	(segment
-		(start 234.49 93.2)
-		(end 234.49 92.74)
-		(width 0.3)
-		(layer "F.Cu")
-		(net "+3.3V")
-	)
-	(segment
 		(start 162.387658 93.565328)
 		(end 161.013494 93.565328)
@@
 		(start 153.94 64.5)
 		(end 153.94 61.81)
-		(width 0.2)
+		(width 0.5)
 		(layer "F.Cu")
 		(net "+3.3V")
@@
 		(start 156.48 64.5)
 		(end 156.48 61.77)
-		(width 0.2)
+		(width 0.5)
 		(layer "F.Cu")
 		(net "+3.3V")
@@
 		(layer "F.Cu")
 		(net "+3.3V")
-	)
-	(segment
-		(start 234.49 92.74)
-		(end 231 89.25)
-		(width 0.3)
-		(layer "F.Cu")
-		(net "+3.3V")

Commit message: last version
Parts:
- C22: value 1u -> 1µ
- C28: footprint Capacitor_SMD:C_0402_1005Metric -> Capacitor_SMD:C_0603_1608Metric
- moved C28 0.29 mm to (234.8, 96.8)
Changed lines of the file:
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@@
 		)
 	)
-	(footprint "Capacitor_SMD:C_0402_1005Metric"
+	(footprint "Capacitor_SMD:C_0603_1608Metric"
 		(layer "F.Cu")
-		(at 235 96.6)
-		(descr "Capacitor SMD 0402 (1005 Metric), square (rectangular) end terminal, IPC-7351 nominal, (Body size source: IPC-SM-782 page 76, https://www.pcb-3d.com/wordpress/wp-content/uploads/ipc-sm-782a_amendment_1_and_2.pdf)")
+		(at 234.75 96.75)
+		(descr "Capacitor SMD 0603 (1608 Metric), square (rectangular) end terminal, IPC-7351 nominal, (Body size source: IPC-SM-782 page 76, https://www.pcb-3d.com/wordpress/wp-content/uploads/ipc-sm-782a_amendment_1_and_2.pdf)")
 		(tags "capacitor")
 		(property "Reference" "C28"
-			(at -2.6 0 0)
+			(at 0 -1.43 0)
 			(layer "F.SilkS")
 			(effects
@@
 		)
 		(property "Value" "4,7u"
-			(at 0 1.16 0)
+			(at 0 1.43 0)
 			(layer "F.Fab")
 			(effects
@@
 		(duplicate_pad_numbers_are_jumpers no)
 		(fp_line
-			(start -0.107836 -0.36)
-			(end 0.107836 -0.36)
+			(start -0.14058 -0.51)
+			(end 0.14058 -0.51)
 			(stroke
 				(width 0.12)
@@
 		)
 		(fp_line
-			(start -0.107836 0.36)
-			(end 0.107836 0.36)
+			(start -0.14058 0.51)
+			(end 0.14058 0.51)
 			(stroke
 				(width 0.12)
@@
 		)
 		(fp_rect
-			(start -0.91 -0.46)
-			(end 0.91 0.46)
+			(start -1.48 -0.73)
+			(end 1.48 0.73)
 			(stroke
 				(width 0.05)
@@
 		)
 		(fp_rect
-			(start -0.5 -0.25)
-			(end 0.5 0.25)
+			(start -0.8 -0.4)
+			(end 0.8 0.4)
 			(stroke
 				(width 0.1)
@@
 			(effects
 				(font
-					(size 0.25 0.25)
-					(thickness 0.04)
+					(size 0.4 0.4)
+					(thickness 0.06)
 				)
 			)
 		)
 		(pad "1" smd roundrect
-			(at -0.48 0)
-			(size 0.56 0.62)
+			(at -0.775 0)
+			(size 0.9 0.95)
 			(layers "F.Cu" "F.Mask" "F.Paste")
 			(roundrect_rratio 0.25)
@@
 		)
 		(pad "2" smd roundrect
-			(at 0.48 0)
-			(size 0.56 0.62)
+			(at 0.775 0)
+			(size 0.9 0.95)
 			(layers "F.Cu" "F.Mask" "F.Paste")
 			(roundrect_rratio 0.25)
@@
 		)
 		(embedded_fonts no)
-		(model "${KICAD10_3DMODEL_DIR}/Capacitor_SMD.3dshapes/C_0402_1005Metric.step"
+		(model "${KICAD10_3DMODEL_DIR}/Capacitor_SMD.3dshapes/C_0603_1608Metric.step"
 			(offset
 				(xyz 0 0 0)
@@
 			)
 		)
-		(property "Value" "1u"
+		(property "Value" "1µ"
 			(at 0 1.16 90)
 			(layer "F.Fab")
@@
 	)
 	(segment
+		(start 235.675 96.6)
+		(end 235.525 96.75)
+		(width 0.5)
+		(layer "F.Cu")
+		(net "+3.3V")
+	)
+	(segment
 		(start 150.403806 86.510408)
 		(end 150.332107 86.582107)
@@
 	)
 	(segment
-		(start 235.48 96.6)
-		(end 238.72 96.6)
-		(width 0.5)
-		(layer "F.Cu")
-		(net "+3.3V")
-	)
-	(segment
 		(start 149.7 101.62)
 		(end 151.031612 101.62)
@@
 	)
 	(segment
+		(start 238.72 96.6)
+		(end 235.675 96.6)
+		(width 0.5)
+		(layer "F.Cu")
+		(net "+3.3V")
+	)
+	(segment
 		(start 183.910589 84.089411)
 		(end 183.25 84.75)
@@
 	)
 	(via
-		(at 235.48 96.6)
-		(size 0.6)
-		(drill 0.3)
-		(layers "F.Cu" "B.Cu")
-		(net "+3.3V")
-	)
-	(via
 		(at 185.25 98.25)
 		(size 0.6)
@@
 		(size 0.6)
 		(drill 0.3)
+		(layers "F.Cu" "B.Cu")
+		(net "+3.3V")
+	)
+	(via
+		(at 235.48 96.6)
+		(size 0.6)
+		(drill 0.3)

Commit message: last version
Parts:
- moved C27 0.84 mm to (234.8, 98.0)
Routing:
- net +3.3V: track 107.3 -> 108.5 mm, vias 27 -> 26
Changed lines of the file:
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@@
 	(footprint "Capacitor_SMD:C_0402_1005Metric"
 		(layer "F.Cu")
-		(at 235 98.8 180)
+		(at 234.75 98 180)
 		(descr "Capacitor SMD 0402 (1005 Metric), square (rectangular) end terminal, IPC-7351 nominal, (Body size source: IPC-SM-782 page 76, https://www.pcb-3d.com/wordpress/wp-content/uploads/ipc-sm-782a_amendment_1_and_2.pdf)")
 		(tags "capacitor")
@@
 		(tags "capacitor")
 		(property "Reference" "C28"
-			(at 0 -1.43 0)
+			(at -3 0 0)
 			(layer "F.SilkS")
 			(effects
@@
 	)
 	(segment
-		(start 235.48 98.8)
-		(end 235.48 98.92)
-		(width 0.3)
-		(layer "F.Cu")
-		(net "+3.3V")
-	)
-	(segment
 		(start 162.239411 99.939411)
 		(end 162.928822 99.25)
@@
 	)
 	(segment
+		(start 235.525 97.705)
+		(end 235.23 98)
+		(width 0.5)
+		(layer "F.Cu")
+		(net "+3.3V")
+	)
+	(segment
 		(start 150.02 91.25)
 		(end 150.02 91.2)
@@
 	)
 	(segment
+		(start 235.525 96.75)
+		(end 235.525 97.705)
+		(width 0.5)
+		(layer "F.Cu")
+		(net "+3.3V")
+	)
+	(segment
 		(start 169 101.165833)
 		(end 169 100.75)
@@
 	)
 	(via
-		(at 235.48 98.92)
-		(size 0.6)
-		(drill 0.3)
-		(layers "F.Cu" "B.Cu")
-		(net "+3.3V")
-	)
-	(via
 		(at 175 106.75)
 		(size 0.6)
@@
 	(segment
 		(start 237.300001 97.699999)
+		(end 238.719999 97.699999)
+		(width 0.2)
+		(layer "F.Cu")
+		(net "SD_CK")
+	)
+	(segment
+		(start 236.5 98)
 		(end 237 98)
 		(width 0.2)
@@
 	)
 	(segment
-		(start 238.719999 97.699999)
+		(start 237 98)
 		(end 237.300001 97.699999)
 		(width 0.2)
@@
 	)
 	(via
-		(at 237 98)
+		(at 236.5 98)
 		(size 0.6)
 		(drill 0.3)
@@
 	)
 	(segment
-		(start 203.25 90.5)
+		(start 236.5 98)
 		(end 210.75 98)
 		(width 0.2)
@@
 	)
 	(segment
-		(start 181.5 90.5)
+		(start 210.75 98)
 		(end 203.25 90.5)
 		(width 0.2)
@@
 	)
 	(segment
-		(start 210.75 98)
-		(end 237 98)
+		(start 203.25 90.5)
+		(end 181.5 90.5)
 		(width 0.2)
 		(layer "B.Cu")

Commit message: last version
Parts:
- SW1: renamed from NRST_BTN-1; value switch -> ~
- SW2: renamed from BOOT_BTN-2; value switch -> ~
Changed lines of the file:
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@@
 		(layer "F.Cu")
 		(at 201.48 102.9 180)
-		(property "Reference" "NRST_BTN-1"
+		(property "Reference" "SW1"
 			(at -4.5 -0.1 0)
 			(layer "F.SilkS")
@@
 			)
 		)
-		(property "Value" "switch"
+		(property "Value" "~"
 			(at 0 4.74 0)
 			(layer "F.Fab")
@@
 			(size 1.05 1.15)
 			(layers "F.Cu" "F.Mask" "F.Paste")
-			(net "unconnected-(NRST_BTN-1-Pad1)")
+			(net "unconnected-(SW1-Pad1)")
 			(pinfunction "1_1")
 			(pintype "unspecified+no_connect")
@@
 			(size 1.05 1.15)
 			(layers "F.Cu" "F.Mask" "F.Paste")
-			(net "unconnected-(NRST_BTN-1-Pad2')")
+			(net "unconnected-(SW1-Pad2')")
 			(pinfunction "2'_2'")
 			(pintype "unspecified+no_connect")
@@
 			)
 		)
-		(property "LCSC Part" "C102683"
+		(property "LCSC Part" "C11702"
 			(at 0 0 0)
 			(unlocked yes)
@@
 		(layer "F.Cu")
 		(at 201.5 107.3)
-		(property "Reference" "BOOT_BTN-2"
+		(property "Reference" "SW2"
 			(at 4.7 -0.8 0)
 			(layer "F.SilkS")
@@
 			)
 		)
-		(property "Value" "switch"
+		(property "Value" "~"
 			(at 0 4.74 0)
 			(layer "F.Fab")
@@
 			(size 1.05 1.15)
 			(layers "F.Cu" "F.Mask" "F.Paste")
-			(net "unconnected-(BOOT_BTN-2-Pad1')")
+			(net "unconnected-(SW2-Pad1')")
 			(pinfunction "1'_1'")
 			(pintype "unspecified+no_connect")
@@
 			(size 1.05 1.15)
 			(layers "F.Cu" "F.Mask" "F.Paste")
-			(net "unconnected-(BOOT_BTN-2-Pad2)")
+			(net "unconnected-(SW2-Pad2)")
 			(pinfunction "2_2")
 			(pintype "unspecified+no_connect")
@@
 			)
 		)
-		(property "LCSC Part" "C102683"
+		(property "LCSC Part" "C11702"
 			(at 0 0 0)
 			(unlocked yes)

Commit message: last version
Parts:
- added G***: LOGO, logo:logo_feuille, B.Cu at (170.0, 88.2)
- moved H2 1.05 mm to (170.5, 57.2)
Routing:
- net +5V: track 14.0 -> 13.4 mm
Other:
- board text added: "3.3V"
- board text added: "5V"
- board text added: "Boot"
- board text added: "EL-STDBY"
- board text added: "FILS"
- board text added: "GND"
- board text added: "GNSS"
- board text added: "L'INDEX STELLAIRE"
- board text added: "Reset"
- board text added: "SCREEN/JOY/ALIM"
- board text added: "TACTIL"
- board text added: "TMC2209 AZ - 11"
- board text added: "TMC2209 EL - 10"
