File: Hardware/PCB/PCB_Mere/KiCad/PCB_Mere_V1.kicad_pcb (KiCad board)
At the start: 4 copper layers, 113.4 x 80.1 mm, 80 parts, among them CN1 FTSH-107-01-L-DV-K-A, CN2 B4B-PH-K-S_GNSS, U1 STM32H723ZGT6, U2 LORA1276-C1-868MHZ, U3 ESP32C3-SUPERMINI, U4 BNO055, U5 B8B-PH-K-S-_TACTIL, U6 B8B-PH-K-S_FILS, U7 B10B-PH-K-S-_SCRN/JOY/ALIM, U8 A-SP1102AR6GHC-A01-2C, X1 X322525MOB4SI, X2 X701532768KGD4GI

Commit message: last version + Ajout du PCB Fils FINI?
Parts:
- moved G*** 2.51 mm to (170.2, 85.8)
Routing:
- net TMC2209_AZ_INDEX_GPIO_Input: track 27.1 -> 27.9 mm
- net NRST_STM: track 83.1 -> 83.7 mm
- net LED1_ETAT_GPIO_Output: track 31.9 -> 31.3 mm
- net TMC2209_AZ_STDBY_GPIO_Output: track 40.9 -> 41.2 mm, vias 1 -> 2
- net GND: vias 193 -> 198
Other:
- board text added: "Carte Mère"
- board text added: "L'INDEX STELLAIRE : L'ASTROLAB"
- board text removed: "L'INDEX STELLAIRE"
