File: Hardware/PCB/PCB_Mere/KiCad/Composant_Mere.kicad_sch (KiCad schematic)
At the start: 28 parts, among them CN1 FTSH-107-01-L-DV-K-A, U2 LORA1276-C1-868MHZ, U3 ESP32C3-SUPERMINI, U4 BNO055

Commit message: push du kicad
Connections:
- net +3.3V: no longer U4.28 (VDDIO)
- net ESP32_UART7_RX: now also U3.2 (GPIO6); no longer U3.1 (GPIO5)
- net ESP32_UART7_TX: now also U3.1 (GPIO5); no longer U3.2 (GPIO6)
Other:
- moved on the sheet: C23, C25, C26

Commit message: Dernière version Schématique
Parts:
- added H2, H4, H5: MountingHole_Pad, footprint:MountingHole_3.2mm_M3, symbol Mechanical:MountingHole_Pad
- added R15: 330, Resistor_SMD:R_0201_0603Metric, symbol Device:R_Small
- added R16: 1k, Resistor_SMD:R_0201_0603Metric, symbol Device:R_Small
- added U8: A-SP1102AR6GHC-A01-2C, EasyEDA:LED-SMD_4P-L3.0-W1.5_A-SP1102AR6GHC-A01-2C, symbol EasyEDA:A-SP1102AR6GHC-A01-2C
- C22: footprint (none) -> Capacitor_SMD:C_0201_0603Metric; LCSC Part (none) -> C52923
- C23: footprint (none) -> Capacitor_SMD:C_0201_0603Metric; LCSC Part (none) -> C18164575
- C24, C27, C33, C35: footprint (none) -> Capacitor_SMD:C_0201_0603Metric; LCSC Part (none) -> C49062
- C25, C26: footprint (none) -> Capacitor_SMD:C_0201_0603Metric; LCSC Part (none) -> C76924
- C28: footprint (none) -> Capacitor_SMD:C_0201_0603Metric; LCSC Part (none) -> C19666
- C29: footprint (none) -> Capacitor_SMD:C_0402_1005Metric; LCSC Part (none) -> C15195
- C34: value 47k -> 100n; footprint (none) -> Capacitor_SMD:C_0201_0603Metric; LCSC Part (none) -> C49062
- R10, R11, R2, R3, R4: footprint (none) -> Resistor_SMD:R_0201_0603Metric; LCSC Part (none) -> C100140
- R12, R13, R8, R9: footprint (none) -> Resistor_SMD:R_0201_0603Metric; LCSC Part (none) -> C100126
- R5, R6, R7: footprint (none) -> Resistor_SMD:R_0201_0603Metric; LCSC Part (none) -> C19420386
Connections:
- net +3.3V: now also R16.1
- net GND: now also H2.1, H4.1, H5.1, U8.3 (K), U8.4 (K)
- new net: R16.2, U8.1 (A)
- new net: R15.2, U8.2 (A)
- new net LED1_ETAT_GPIO_Output: R15.1
- no-connect marks 17 -> 36
Other:
- note added: "G"
- note added: "LED Etat"
- note added: "PTS d'encrage"
- note added: "R"

Commit message: Nouvelles empreintes de mounting holes et plusieurs court circuits retirés du schematic
Parts:
- H2, H4, H5: footprint footprint:MountingHole_3.2mm_M3 -> MountingHole:MountingHole_3.2mm_M3_DIN965_Pad_TopBottom
Changed lines of the file:
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@@
 			)
 		)
-		(property "Footprint" "footprint:MountingHole_3.2mm_M3"
+		(property "Footprint" "MountingHole:MountingHole_3.2mm_M3_DIN965_Pad_TopBottom"
 			(at 147.32 265.43 0)
 			(hide yes)
@@
 	)
 	(symbol
-		(lib_id "power:GND")
-		(at 148.59 200.66 0)
-		(unit 1)
-		(body_style 1)
-		(exclude_from_sim no)
-		(in_bom yes)
-		(on_board yes)
-		(in_pos_files yes)
-		(dnp no)
-		(fields_autoplaced yes)
-		(property "Reference" "#PWR017"
-			(at 148.59 207.01 0)
-			(hide yes)
-			(show_name no)
-			(do_not_autoplace no)
-			(effects
-				(font
-					(size 1.27 1.27)
-				)
-			)
-		)
-		(property "Value" "GND"
-			(at 151.13 201.9299 0)
-			(show_name no)
-			(do_not_autoplace no)
-			(effects
-				(font
-					(size 1.27 1.27)
-				)
-				(justify left)
-			)
-		)
-		(property "Footprint" ""
-			(at 148.59 200.66 0)
-			(hide yes)
-			(show_name no)
-			(do_not_autoplace no)
-			(effects
-				(font
-					(size 1.27 1.27)
-				)
-			)
-		)
-		(property "Datasheet" ""
-			(at 148.59 200.66 0)
-			(hide yes)
-			(show_name no)
-			(do_not_autoplace no)
-			(effects
-				(font
-					(size 1.27 1.27)
-				)
-			)
-		)
-		(property "Description" "Power symbol creates a global label with name \"GND\" , ground"
-			(at 148.59 200.66 0)
-			(hide yes)
-			(show_name no)
-			(do_not_autoplace no)
-			(effects
-				(font
-					(size 1.27 1.27)
-				)
-			)
-		)
-		(pin "1"
-		)
-		(instances
-			(project "PCB_Mere_V1"
-				(path "/d2ac468b-9b53-4c3c-b006-996db3620a48/46fcd7a3-97be-4e38-b68a-1e4eb53a4357"
-					(reference "#PWR017")
-					(unit 1)
-				)
-			)
-		)
-	)
-	(symbol
 		(lib_id "power:+3.3V")
 		(at 82.55 203.2 90)
@@
 			)
 		)
-		(property "Footprint" "footprint:MountingHole_3.2mm_M3"
+		(property "Footprint" "MountingHole:MountingHole_3.2mm_M3_DIN965_Pad_TopBottom"
 			(at 170.18 265.43 0)
 			(hide yes)
@@
 			)
 		)
-		(property "Footprint" "footprint:MountingHole_3.2mm_M3"
+		(property "Footprint" "MountingHole:MountingHole_3.2mm_M3_DIN965_Pad_TopBottom"
 			(at 195.58 265.43 0)
 			(hide yes)

Commit message: avancement schematic fils
Changed lines of the file:
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@@
 		)
 		(property "Value" "10k"
-			(at 327.66 69.596 90)
+			(at 327.914 69.088 90)
 			(show_name no)
 			(do_not_autoplace no)

Commit message: Push PCB_Mère avancement routage
Parts:
- removed C35: 100n, Capacitor_SMD:C_0201_0603Metric, symbol Device:C_Small
- added D1: SS34_C8678, EasyEDA:SMA_L4.3-W2.6-LS5.2-RD, symbol EasyEDA:SS34_C8678
- added X2: X701532768KGD4GI, EasyEDA:MC-146_4P-L6.7-W1.5-P0.85-BL, symbol EasyEDA:X701532768KGD4GI
- C22, C24, C25, C26, C27, C28, C33, C34: footprint Capacitor_SMD:C_0201_0603Metric -> Capacitor_SMD:C_0402_1005Metric
- C23: value 120n -> 100n; footprint Capacitor_SMD:C_0201_0603Metric -> Capacitor_SMD:C_0402_1005Metric
- R10, R11, R12, R13, R15, R16, R2, R3, R4, R5, R6, R7, R8, R9: footprint Resistor_SMD:R_0201_0603Metric -> Resistor_SMD:R_0402_1005Metric
Connections:
- net +3.3V: now also U4.28 (VDDIO); no longer U3.14 (3V3)
- net +5V: now also D1.2 (A); no longer C34.2, U3.16 (5V)
- net GND: now also X2.3 (GND), X2.4 (OSC2)
- net at C26.2, U4.26 (XOUT32): now also X2.2 (GND)
- net LoRa_NRST_STM_GPIO_Output: now reaches U2.6 (NRESET)
- net at C25.2, U4.27 (XIN32): now also X2.1 (OSC1)
- new net: C34.2, D1.1 (K), U3.16 (5V)
Other:
- moved on the sheet: C25, C26

Commit message: last version
Parts:
- C23: LCSC Part C18164575 -> C1525
- C24, C27, C33, C34: LCSC Part C49062 -> C1525
- C25, C26: LCSC Part C76924 -> C1555
- R10, R11, R2, R3, R4: LCSC Part C100140 -> C25792
- R12, R13, R8, R9: LCSC Part C100126 -> C25744
- R15: LCSC Part 320833 -> C25104
- R16: LCSC Part C102683 -> C11702
- R5, R6, R7: LCSC Part C19420386 -> C25879

Commit message: last version
Parts:
- C22: value 1u -> 1µ
- C28: footprint Capacitor_SMD:C_0402_1005Metric -> Capacitor_SMD:C_0603_1608Metric
Changed lines of the file:
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@@
 			)
 		)
-		(property "Value" "1u"
+		(property "Value" "1µ"
 			(at 90.17 216.154 90)
 			(show_name no)
@@
 			)
 		)
-		(property "Footprint" "Capacitor_SMD:C_0402_1005Metric"
+		(property "Footprint" "Capacitor_SMD:C_0603_1608Metric"
 			(at 289.56 49.53 0)
 			(hide yes)
