File: Hardware/PCB/PCB_Pere/KiCad_Pere/PCB_Pere_V1/Driver_elevation.kicad_sch (KiCad schematic)
At the start: 0 parts

Commit message: Routage toujours en attente oui je sais ça prend 10 000  ans mais it is what is
Parts:
- added C35, C41, C43: 2.2uF, EasyEDA:C1206, symbol EasyEDA:TCC1206X7R225K500FT
- added C36, C37, C38, C42, C44, C45, C46: 100nF, EasyEDA:C0603, symbol EasyEDA:CC0603KRX7R9BB104
- added C39: 22nF, EasyEDA:C0805, symbol EasyEDA:CL21B223KBANNNC
- added LED3: Yellow, EasyEDA:LED0805-R-RD, symbol EasyEDA:17-21SUYC_TR8
- added R12: 1kΩ, EasyEDA:R0603, symbol EasyEDA:0603WAF1001T5E
- added R16: TC33X-2-103E, EasyEDA:RES-ADJ-SMD_3P-L3.0-W3.8-P1.75-BR, symbol EasyEDA:TC33X-2-103E
- added R17: 10k, EasyEDA:R0603, symbol EasyEDA:0603WAF1002T5E
- added R18: 1KΩ, EasyEDA:R0603, symbol EasyEDA:0603WAF1001T5E
- added R19, R8: 100kΩ, EasyEDA:R0603, symbol EasyEDA:0603WAF1003T5E
- added R20, R21: 120mΩ, EasyEDA:R2512, symbol EasyEDA:25121WF120LT4E
- added U6: 8132H-10.000NL33DTL, EasyEDA:OSC-SMD_4P-L3.2-W2.5-BL, symbol EasyEDA:8132H-10.000NL33DTL
- added U7: TMC2209-LA-T, EasyEDA:QFN-28_L5.0-W5.0-P0.50-BL-EP, symbol EasyEDA:TMC2209-LA-T
Connections:
- new net: LED3.1 (+), R12.1
- new net: U6.3 (OUTPUT_RF), U7.13 (CLK)
- new net: C35.1, R17.2, U7.8 (5VOUT)
- new net: C39.1, U7.5 (CPI)
- new net: C39.2, U7.4 (CPO)
- new net: R16.3, R17.1
- new net: C37.1, U7.6 (VCP)
- new net +20V: C37.2, C38.2, C41.2, C42.2, C43.2, U7.22 (VS), U7.28 (VS)
- new net +3V3: C36.1, C44.2, U6.4 (VCC), U7.15 (VCC_IO)
- new net BRA: C46.2, R21.2, U7.27 (BRB)
- new net BRB: C45.2, R20.2, U7.23 (BRA)
- new net DIAG: R12.2, U7.11 (DIAG)
- new net DIR: U7.19 (DIR)
- new net ENN: U7.2 (ENN)
- new net GND: C35.2, C36.2, C38.1, C41.1, C42.1, C43.1, C44.1, C45.1, C46.1, LED3.2 (-), R16.1, R19.1, R20.1, R21.1, R8.1, U6.2 (GND), U7.18 (GND), U7.29 (EP), U7.3 (GND)
- new net Index: U7.12 (INDEX)
- new net MS1: U7.9 (MS1_AD0)
- new net MS2: U7.10 (MS2_AD1)
- new net OA1: U7.24 (OA1)
- new net OA2: U7.21 (OA2)
- new net OB1: U7.26 (OB1)
- new net OB2: U7.1 (OB2)
- new net STDBY: R19.2, U7.20 (STDBY)
- new net STEP: U7.16 (STEP)
- new net Spread: R8.2, U7.7 (SPREAD)
- new net UART_RX: R18.2, U7.14 (PDN_UART)
- new net UART_TX: R18.1
- new net VREF: R16.2, U7.17 (VREF)
- no-connect marks 0 -> 2
Other:
- note added: "Driver Elévation"
- note added: "Le Vref est réglable entre 0 et 2.5V pour pouvoir limiter le courant en mode autonome. 0Ohms -> 0V 10kOhms -> 2.5V : Ampérage maximal : 1.64A RMS (moteur 1.7A) Le réglage du potentiomètre n'est pas nécessaire avec l'utilisation de l'UART mais il reste possible d'utiliser Vref dans les paramètres de l'UART"
- note added: "Le crystal thermorégulé est de 10MHz, tandis que la valeur par défaut du TMC2209 est de 12MHz, ce décalage doit tre compensé dans le paramètrage de l'UART"
- note added: "Reste à faire : (liste finie) ajouter des condensateurs en entrée de puissance voir si on a besoin du standby + ajouter pulldown keskeusé keut le 5Vout ? Voir comment gérer les sense resistor avec Vref et les BRB"
