File: Hardware/PCB/PCB_Pere/KiCad_Pere/PCB_Pere_V1/Driver_azimutal.kicad_sch (KiCad schematic)
At the start: 11 parts, among them U1 TMC2209-LA-T, X2 12 MHz

Commit message: mise à jour PCB père
Parts:
- added R1, R2: 120mΩ, EasyEDA:R2512, symbol EasyEDA:25121WF120LT4E
- added R4: 100kΩ, EasyEDA:R0603, symbol EasyEDA:0603WAF1003T5E
- C12: renamed from C1; value RVT1H331M1010 -> 330uF
- C23: renamed from C2; value RVT1H331M1010 -> 330uF
- R5: renamed from R2; value 1KΩ -> 1kΩ
- renumbered C3 to C10, C5 to C11, C6 to C24, C4 to C9, LED1 to LED2, R1 to R10, U1 to U2, X2 to X3
Connections:
- net GND: now also R1.1, R2.1, R4.1
- net Spread: now also U2.7 (SPREAD), R4.2
- net +20V: now reaches C12.1
- net +20V: now also C10.2, C23.1, C9.2, U2.22 (VS), U2.28 (VS)
- net STDBY: now reaches U2.20 (STDBY)
- net BRB: now reaches U2.23 (BRA)
- net BRB: now also R2.2
- net BRA: now reaches U2.27 (BRB)
- net BRA: now also R1.2
- no-connect marks 1 -> 2
Other:
- note removed: "prende passe inductance pour les résistances de Rsa et RSB 0.5W, 1206"

Commit message: Routage toujours en attente oui je sais ça prend 10 000  ans mais it is what is
Parts:
- removed C12, C23: 330uF, EasyEDA:CAP-SMD_BD10.0-L10.3-W10.3-LS11.0-FD, symbol EasyEDA:RVT1H331M1010
- removed X3: 12 MHz, EasyEDA:CRYSTAL-SMD_4P-L3.2-W2.5-BL, symbol EasyEDA:X322512MSB4SI
- added C12, C25, C26, C30: 100nF, EasyEDA:C0603, symbol EasyEDA:CC0603KRX7R9BB104
- added C2, C4, C40: 2.2uF, EasyEDA:C1206, symbol EasyEDA:TCC1206X7R225K500FT
- added R14: TC33X-2-103E, EasyEDA:RES-ADJ-SMD_3P-L3.0-W3.8-P1.75-BR, symbol EasyEDA:TC33X-2-103E
- added R15: 10k, EasyEDA:R0603, symbol EasyEDA:0603WAF1002T5E
- added R3: 100kΩ, EasyEDA:R0603, symbol EasyEDA:0603WAF1003T5E
- added U4: 8132H-10.000NL33DTL, EasyEDA:OSC-SMD_4P-L3.2-W2.5-BL, symbol EasyEDA:8132H-10.000NL33DTL
Connections:
- net +20V: now also C12.2, C4.2, C40.2
- net +3V3: now also C30.1, U4.4 (VCC)
- net BRA: now also C26.2
- net BRB: now also C25.2
- net GND: now also C12.1, C2.2, C25.1, C26.1, C30.2, C4.1, C40.1, R14.1, R3.1, U4.2 (GND)
- net STDBY: now also R3.2
- net at U2.13 (CLK): now also U4.3 (OUTPUT_RF)
- net VREF: now reaches U2.17 (VREF)
- net VREF: now also R14.2
- net at U2.8 (5VOUT): now also C2.1, R15.2
- new net: R14.3, R15.1
Other:
- note added: "Driver Elévation"
- note added: "Le Vref est réglable entre 0 et 2.5V pour pouvoir limiter le courant en mode autonome. 0Ohms -> 0V 10kOhms -> 2.5V : Ampérage maximal : 1.64A RMS (moteur 1.7A) Le réglage du potentiomètre n'est pas nécessaire avec l'utilisation de l'UART mais il reste possible d'utiliser Vref dans les paramètres de l'UART"
- note removed: "Led jaune de debug en plus d'un signal envoyé à la stm"
- moved on the sheet: C10, C9, LED2, R4, R5

Commit message: pcb père quasi fini
Connections:
- net BRA: now also C25.2, R2.2, U2.23 (BRA); no longer C26.2, R1.2, U2.27 (BRB)
- net BRB: now also C26.2, R1.2, U2.27 (BRB); no longer C25.2, R2.2, U2.23 (BRA)
Changed lines of the file:
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@@
 		)
 	)
-	(hierarchical_label "BRB"
+	(hierarchical_label "BRA"
 		(shape output)
 		(at 186.69 96.52 0)
@@
 		)
 	)
-	(hierarchical_label "BRA"
+	(hierarchical_label "BRB"
 		(shape output)
 		(at 204.47 86.36 0)
