File: Hardware/PCB/PCB_Pere/KiCad_Pere/PCB_Pere_V1/PCB_Pere_V1.kicad_pcb (KiCad board)
At the start: 2 copper layers, 7 parts, among them CN2 B4B-PH-K-S, U1 TMC2209-LA-T, U3 LMR51625XDDCR_C44750835, U4 LMR51625XDDCR_C44750835, X2 X322512MSB4SI

Commit message: mise à jour PCB père
Parts:
- removed U4: LMR51625XDDCR_C44750835, EasyEDA:SOT-23-6_L2.9-W1.6-P0.95-LS2.9-BL
- added C1: 330uF, EasyEDA:CAP-SMD_BD10.0-L10.3-W10.3-LS11.0-FD, F.Cu at (154.8, 80.5)
- added C10: 100nF, EasyEDA:C0603, F.Cu at (137.0, 94.1)
- added C11: 22nF, EasyEDA:C0805, F.Cu at (143.0, 86.8)
- added C12: 330uF, EasyEDA:CAP-SMD_BD10.0-L10.3-W10.3-LS11.0-FD, F.Cu at (127.8, 80.5)
- added C13: 33uF, EasyEDA:C1812, F.Cu at (151.4, 54.9)
- added C14: 33uF, EasyEDA:C1812, F.Cu at (151.4, 60.0)
- added C15: 100nF, EasyEDA:C0603, F.Cu at (168.6, 53.7)
- added C16: 100nF, EasyEDA:C0603, F.Cu at (168.6, 56.4)
- added C17: 33uF, EasyEDA:C1812, F.Cu at (151.4, 65.0)
- added C18: 33uF, EasyEDA:C1812, F.Cu at (151.4, 70.1)
- added C19: 100nF, EasyEDA:C0603, F.Cu at (168.6, 59.0)
- added C2: 330uF, EasyEDA:CAP-SMD_BD10.0-L10.3-W10.3-LS11.0-FD, F.Cu at (154.8, 92.1)
- added C20: 100nF, EasyEDA:C0603, F.Cu at (168.6, 61.7)
- added C21: 22nF, EasyEDA:C0805, F.Cu at (127.0, 65.5)
- added C22: 22nF, EasyEDA:C0805, F.Cu at (127.0, 68.4)
- added C23: 330uF, EasyEDA:CAP-SMD_BD10.0-L10.3-W10.3-LS11.0-FD, F.Cu at (127.8, 92.1)
- added C24: 100nF, EasyEDA:C0603, F.Cu at (137.0, 96.8)
- added C3: 100nF, EasyEDA:C0603, F.Cu at (164.0, 91.4)
- added C4: 100nF, EasyEDA:C0603, F.Cu at (164.0, 94.1)
- added C5: 22nF, EasyEDA:C0805, F.Cu at (170.0, 86.8)
- added C6: 100nF, EasyEDA:C0603, F.Cu at (164.0, 96.8)
- added C7: 2.2uF, EasyEDA:C1206, F.Cu at (141.5, 64.3)
- added C8: 2.2uF, EasyEDA:C1206, F.Cu at (141.5, 67.6)
- added C9: 100nF, EasyEDA:C0603, F.Cu at (137.0, 91.4)
- added CN3: B4B-PH-K-S, EasyEDA:CONN-TH_B4B-PH-K-S, F.Cu at (160.9, 61.7)
- added L1: 10uH, EasyEDA:IND-SMD_L5.4-W5.2_FAUL0530-100MT, F.Cu at (141.9, 59.4)
- added L4: 15uF, EasyEDA:IND-SMD_L7.0-W6.6_MCW-0650-220, F.Cu at (129.1, 60.1)
- added LED1: Yellow, EasyEDA:LED0805-R-RD, F.Cu at (164.9, 83.7)
- added LED2: Yellow, EasyEDA:LED0805-R-RD, F.Cu at (137.8, 83.7)
- added R1: 1KΩ, EasyEDA:R0603, F.Cu at (168.0, 91.3)
- added R1: 120mΩ, EasyEDA:R2512, F.Cu at (138.5, 37.5)
- added R10: 1KΩ, EasyEDA:R0603, F.Cu at (141.0, 96.3)
- added R2: 120mΩ, EasyEDA:R2512, F.Cu at (138.5, 42.6)
- added R2: 1KΩ, EasyEDA:R0603, F.Cu at (168.0, 93.8)
- added R3: 100kΩ, EasyEDA:R0603, F.Cu at (168.0, 96.3)
- added R4: 100kΩ, EasyEDA:R0603, F.Cu at (141.0, 91.3)
- added R5: 1kΩ, EasyEDA:R0603, F.Cu at (141.0, 93.8)
- added R6: 53.6kR, EasyEDA:R0603, F.Cu at (122.5, 57.4)
- added R7: 31.6kR, EasyEDA:R0603, F.Cu at (122.5, 59.9)
- added R8: 10.2kR, EasyEDA:R0603, F.Cu at (122.5, 62.3)
- added R9: 10.2kR, EasyEDA:R0603, F.Cu at (122.5, 64.8)
- added U2: TMC2209-LA-T, EasyEDA:QFN-28_L5.0-W5.0-P0.50-BL-EP, F.Cu at (139.0, 77.0)
- added U5: Buck LMR51625, EasyEDA:SOT-23-6_L2.9-W1.6-P0.95-LS2.9-BL, F.Cu at (136.3, 62.7)
- added X3: 12 MHz, EasyEDA:CRYSTAL-SMD_4P-L3.2-W2.5-BL, F.Cu at (137.8, 87.6)
- U3: value LMR51625XDDCR_C44750835 -> Buck LMR51625
- X2: value X322512MSB4SI -> 12 MHz
- moved CN2 53.9 mm to (160.9, 55.9)
- moved U3 50.5 mm to (136.3, 58.3)
- moved U1 47.6 mm to (165.5, 78.1)
- moved H1 39.8 mm to (146.5, 50.5)
- moved H2 39.8 mm to (134.0, 54.3)
- moved X2 37.5 mm to (164.8, 87.6)
Connections:
- U1 pad 10: unconnected-(U1-MS2_AD1-Pad10) -> /Interfaces/Driver Azimutal/MS2
- U1 pad 11: unconnected-(U1-DIAG-Pad11) -> /Interfaces/Driver Azimutal/DIAG
- U1 pad 12: unconnected-(U1-INDEX-Pad12) -> /Interfaces/Driver Azimutal/DIAG
- U1 pad 14: unconnected-(U1-PDN_UART-Pad14) -> /Interfaces/Driver Azimutal/UART_RX
- U1 pad 16: unconnected-(U1-STEP-Pad16) -> /Interfaces/Driver Azimutal/STEP
- U1 pad 19: unconnected-(U1-DIR-Pad19) -> /Interfaces/Driver Azimutal/DIAG
- U1 pad 2: unconnected-(U1-ENN-Pad2) -> /Interfaces/Driver Azimutal/DIAG
- U1 pad 20: unconnected-(U1-STDBY-Pad20) -> /Interfaces/Driver Azimutal/STDBY
- U1 pad 22: unconnected-(U1-VS-Pad22) -> Net-(C1-Pad1)
- U1 pad 28: unconnected-(U1-VS-Pad28) -> Net-(C1-Pad1)
- U1 pad 29: unconnected-(U1-EP-Pad29) -> GND
- U1 pad 4: unconnected-(U1-CPO-Pad4) -> Net-(U1-CPO)
- U1 pad 5: unconnected-(U1-CPI-Pad5) -> Net-(U1-CPI)
- U1 pad 6: unconnected-(U1-VCP-Pad6) -> Net-(U1-VCP)
- U1 pad 7: unconnected-(U1-SPREAD-Pad7) -> /Interfaces/Driver Azimutal/Spread
- U1 pad 9: unconnected-(U1-MS1_AD0-Pad9) -> /Interfaces/Driver Azimutal/DIAG
- U3 pad 1: unconnected-(U3-FB-Pad1) -> /Interfaces/FB_3V3
- U3 pad 2: unconnected-(U3-EN-Pad2) -> +20V
- U3 pad 3: unconnected-(U3-VIN-Pad3) -> +20V
- U3 pad 4: unconnected-(U3-GND-Pad4) -> GND
- U3 pad 5: unconnected-(U3-SW-Pad5) -> Net-(U3-SW)
- U3 pad 6: unconnected-(U3-CB-Pad6) -> Net-(U3-CB)

Commit message: Routage toujours en attente oui je sais ça prend 10 000  ans mais it is what is
Parts:
- removed C1: 330uF, EasyEDA:CAP-SMD_BD10.0-L10.3-W10.3-LS11.0-FD
- removed CN2: B4B-PH-K-S, EasyEDA:CONN-TH_B4B-PH-K-S
- removed LED1: Yellow, EasyEDA:LED0805-R-RD
- removed the R1 at (168.0, 91.3)
- removed the R1 at (138.5, 37.5)
- removed the R2 at (138.5, 42.6)
- removed the R2 at (168.0, 93.8)
- removed U1: TMC2209-LA-T, EasyEDA:QFN-28_L5.0-W5.0-P0.50-BL-EP
- removed X2, X3: 12 MHz, EasyEDA:CRYSTAL-SMD_4P-L3.2-W2.5-BL
- added C25: 100nF, EasyEDA:C0603, F.Cu at (178.8, 40.2)
- added C26: 100nF, EasyEDA:C0603, F.Cu at (178.8, 29.3)
- added C27: 330uF, EasyEDA:CAP-SMD_BD10.0-L10.3-W10.3-LS11.0-FD, F.Cu at (183.5, 99.0)
- added C28: 330uF, EasyEDA:CAP-SMD_BD10.0-L10.3-W10.3-LS11.0-FD, F.Cu at (183.5, 88.0)
- added C29: 490pF, EasyEDA:C0603, F.Cu at (194.8, 76.4)
- added C30: 100nF, EasyEDA:C0603, F.Cu at (173.3, 41.8)
- added C31: 490pF, EasyEDA:C0603, F.Cu at (194.9, 110.7)
- added C32: 490pF, EasyEDA:C0603, F.Cu at (194.9, 105.0)
- added C33: 490pF, EasyEDA:C0603, F.Cu at (194.9, 108.8)
- added C34: 490pF, EasyEDA:C0603, F.Cu at (194.9, 106.9)
- added C35: 2.2uF, EasyEDA:C1206, F.Cu at (240.1, 37.5)
- added C36: 100nF, EasyEDA:C0603, F.Cu at (228.8, 33.5)
- added C37: 100nF, EasyEDA:C0603, F.Cu at (228.8, 36.2)
- added C38: 100nF, EasyEDA:C0603, F.Cu at (245.2, 31.1)
- added C39: 22nF, EasyEDA:C0805, F.Cu at (214.0, 26.6)
- added C40: 2.2uF, EasyEDA:C1206, F.Cu at (177.0, 26.0)
- added C41: 2.2uF, EasyEDA:C1206, F.Cu at (224.9, 25.6)
- added C42: 100nF, EasyEDA:C0603, F.Cu at (245.1, 29.6)
- added C43: 2.2uF, EasyEDA:C1206, F.Cu at (240.3, 29.6)
- added C44: 100nF, EasyEDA:C0603, F.Cu at (251.5, 37.5)
- added C45: 100nF, EasyEDA:C0603, F.Cu at (250.3, 43.9)
- added C46: 100nF, EasyEDA:C0603, F.Cu at (256.0, 36.2)
- added CN1: B2B-PH-K-S-GW, EasyEDA:CONN-TH_B2B-PH-K-S, F.Cu at (193.7, 93.5)
- added CN4: B4B-PH-K-S, EasyEDA:CONN-TH_B4B-PH-K-S, F.Cu at (191.1, 108.0)
- added LED3: Yellow, EasyEDA:LED0805-R-RD, F.Cu at (208.4, 36.2)
- added R1: 120mΩ, EasyEDA:R2512, F.Cu at (183.5, 31.2)
- added R11: 47k, EasyEDA:R0603, F.Cu at (158.0, 104.0)
- added R12: 1kΩ, EasyEDA:R0603, F.Cu at (220.2, 34.1)
- added R13: 1KΩ, EasyEDA:R0603, F.Cu at (177.2, 96.1)
- added R14: TC33X-2-103E, EasyEDA:RES-ADJ-SMD_3P-L3.0-W3.8-P1.75-BR, F.Cu at (169.0, 36.7)
- added R15: 10k, EasyEDA:R0603, F.Cu at (169.0, 33.5)
- added R16: TC33X-2-103E, EasyEDA:RES-ADJ-SMD_3P-L3.0-W3.8-P1.75-BR, F.Cu at (241.7, 33.4)
- added R17: 10k, EasyEDA:R0603, F.Cu at (220.2, 36.6)
- added R18: 1KΩ, EasyEDA:R0603, F.Cu at (220.2, 39.1)
- added R19: 100kΩ, EasyEDA:R0603, F.Cu at (220.2, 41.5)
- added R2: 120mΩ, EasyEDA:R2512, F.Cu at (183.5, 38.5)
- added R20: 120mΩ, EasyEDA:R2512, F.Cu at (250.2, 41.1)
- added R21: 120mΩ, EasyEDA:R2512, F.Cu at (256.0, 33.7)
- added TP1: TestPoint, TestPoint:TestPoint_Pad_D2.5mm, F.Cu at (115.9, 84.0)
- added TP2: TestPoint, TestPoint:TestPoint_Pad_D2.5mm, F.Cu at (131.0, 47.5)
- added TP3: TestPoint, TestPoint:TestPoint_Pad_D2.5mm, F.Cu at (131.0, 53.2)
- added TP4: TestPoint, TestPoint:TestPoint_Pad_D2.5mm, F.Cu at (131.0, 59.0)
- added TP5: TestPoint, TestPoint:TestPoint_Pad_D2.5mm, F.Cu at (156.2, 120.9)
- added TP6: TestPoint, TestPoint:TestPoint_Pad_2.5x2.5mm, F.Cu at (155.0, 71.0)
- added TP7: TestPoint, TestPoint:TestPoint_Pad_2.5x2.5mm, F.Cu at (193.5, 87.6)
- added U4: 8132H-10.000NL33DTL, EasyEDA:OSC-SMD_4P-L3.2-W2.5-BL, F.Cu at (170.8, 41.1)
- added U6: 8132H-10.000NL33DTL, EasyEDA:OSC-SMD_4P-L3.2-W2.5-BL, F.Cu at (244.1, 41.7)
- added U7: TMC2209-LA-T, EasyEDA:QFN-28_L5.0-W5.0-P0.50-BL-EP, F.Cu at (247.8, 35.0)
- C12: value 330uF -> 100nF; footprint EasyEDA:CAP-SMD_BD10.0-L10.3-W10.3-LS11.0-FD -> EasyEDA:C0603
- C2: value 330uF -> 2.2uF; footprint EasyEDA:CAP-SMD_BD10.0-L10.3-W10.3-LS11.0-FD -> EasyEDA:C1206
- C23: value 330uF -> 490pF; footprint EasyEDA:CAP-SMD_BD10.0-L10.3-W10.3-LS11.0-FD -> EasyEDA:C0603
- C3, C4: value 100nF -> 2.2uF; footprint EasyEDA:C0603 -> EasyEDA:C1206
- C5: value 22nF -> 490pF; footprint EasyEDA:C0805 -> EasyEDA:C0603
- C6: value 100nF -> 490pF
- R6: value 53.6kR -> 47k
- R7: value 31.6kR -> 9.1k
- R8: value 10.2kR -> 100kΩ
- R9: value 10.2kR -> 15k
- moved R8 123.1 mm to (242.6, 35.6)
- moved H2 83.9 mm to (182.9, 122.5), turned to 180 degrees
- moved C10 74.6 mm to (178.7, 32.2), turned to -90 degrees
- moved C9 71.7 mm to (172.3, 29.1), turned to 90 degrees
- moved R5 71.3 mm to (170.8, 29.1), turned to -90 degrees
- moved C4 68.8 mm to (174.3, 26.1), turned to -90 degrees
- moved C23 68.4 mm to (194.8, 78.3), turned to 180 degrees
- moved C24 68.3 mm to (174.3, 39.6), turned to 180 degrees
- moved LED2 67.2 mm to (171.5, 25.5), turned to -90 degrees
- moved C12 66.8 mm to (178.7, 37.3), turned to 90 degrees
- moved R10 66.0 mm to (165.8, 35.1)
- moved C11 65.6 mm to (175.1, 29.7)
- moved R4 62.9 mm to (165.8, 33.6)
- moved C2 62.1 mm to (168.8, 31.6), turned to 180 degrees
- moved C13 60.7 mm to (160.0, 115.0), turned to 180 degrees
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Connections:
- net /Interfaces/Driver Azimutal1/OA1 renamed /Driver Azimutal1/OA1
- C12 pad 1: +20V -> GND
- C12 pad 2: GND -> +20V
- C2 pad 1: Net-(C1-Pad1) -> Net-(U2-5VOUT)
- C21 pad 1: /Interfaces/FB_3V3 -> /FB_3V3
- C22 pad 1: /Interfaces/FB_5V -> /FB_5V
- C23 pad 1: +20V -> GND
- C23 pad 2: GND -> /Driver Azimutal1/OA2
- C3 pad 1: GND -> Net-(C3-Pad1)
- C3 pad 2: Net-(C1-Pad1) -> +20V
- C4 pad 1: Net-(U1-VCP) -> GND
- C4 pad 2: Net-(C1-Pad1) -> +20V
- C5 pad 1: Net-(U1-CPI) -> /Driver Azimutal1/OB2
- C5 pad 2: Net-(U1-CPO) -> GND
- C6 pad 1: GND -> /Driver Azimutal1/OB1
- C6 pad 2: +3V3 -> GND
- CN3 pad 2: /Interfaces/Driver Azimutal1/OA2 -> /Driver Azimutal1/OA2
- CN3 pad 3: /Interfaces/Driver Azimutal1/OB1 -> /Driver Azimutal1/OB1
- CN3 pad 4: unconnected-(CN3-Pad4) -> /Driver Azimutal1/OB2
- H1 pad 1: unconnected-(H1-Pad1) -> GND
- H1 pad 10: unconnected-(H1-Pad10) -> /Driver Azimutal1/STDBY
- H1 pad 11: unconnected-(H1-Pad11) -> /Driver Azimutal1/STEP
- H1 pad 12: unconnected-(H1-Pad12) -> /Driver Azimutal1/ENN
- H1 pad 13: unconnected-(H1-Pad13) -> /Driver Azimutal1/Spread
- H1 pad 14: unconnected-(H1-Pad14) -> /Driver Azimutal1/DIR
- H1 pad 15: unconnected-(H1-Pad15) -> /Driver Azimutal1/MS1
- H1 pad 16: unconnected-(H1-Pad16) -> /Driver Azimutal1/MS2
- H1 pad 17: unconnected-(H1-Pad17) -> /Driver Azimutal1/DIAG
- H1 pad 18: unconnected-(H1-Pad18) -> /Driver Azimutal1/Index
- H1 pad 19: unconnected-(H1-Pad19) -> /Driver Azimutal1/UART_TX
- H1 pad 2: unconnected-(H1-Pad2) -> +5V
- H1 pad 20: unconnected-(H1-Pad20) -> /Driver Azimutal1/UART_RX
- H1 pad 3: unconnected-(H1-Pad3) -> +3V3
- H1 pad 9: unconnected-(H1-Pad9) -> /STBY_Elevation
- H2 pad 1: unconnected-(H2-Pad1) -> /Driver Elevation/UART_TX
- H2 pad 10: unconnected-(H2-Pad10) -> /Driver Elevation/STEP
- H2 pad 2: unconnected-(H2-Pad2) -> /Driver Elevation/UART_RX
- H2 pad 3: unconnected-(H2-Pad3) -> /Driver Elevation/Index
- H2 pad 4: unconnected-(H2-Pad4) -> /Driver Elevation/DIAG
- H2 pad 5: unconnected-(H2-Pad5) -> /Driver Elevation/MS2
- H2 pad 6: unconnected-(H2-Pad6) -> /Driver Elevation/MS1
- H2 pad 7: unconnected-(H2-Pad7) -> /Driver Elevation/DIR
- H2 pad 8: unconnected-(H2-Pad8) -> /Driver Elevation/Spread
- H2 pad 9: unconnected-(H2-Pad9) -> /Driver Elevation/ENN
- R10 pad 1: /Interfaces/Driver Azimutal1/UART_TX -> /Driver Azimutal1/UART_TX
- R10 pad 2: /Interfaces/Driver Azimutal1/UART_RX -> /Driver Azimutal1/UART_RX
- R3 pad 2: /Interfaces/Driver Azimutal/Spread -> /Driver Azimutal1/STDBY
- R4 pad 2: /Interfaces/Driver Azimutal1/Spread -> /Driver Azimutal1/Spread
- R5 pad 2: /Interfaces/Driver Azimutal1/DIAG -> /Driver Azimutal1/DIAG
- R6 pad 1: /Interfaces/FB_5V -> /FB_5V
- R7 pad 1: /Interfaces/FB_3V3 -> GND
- R7 pad 2: +3V3 -> /FB_5V
- R8 pad 2: /Interfaces/FB_5V -> /Driver Elevation/Spread
- R9 pad 2: /Interfaces/FB_3V3 -> /FB_3V3
- U2 pad 1: /Interfaces/Driver Azimutal1/OB2 -> /Driver Azimutal1/OB2
- U2 pad 10: /Interfaces/Driver Azimutal1/MS2 -> /Driver Azimutal1/MS2
- U2 pad 11: /Interfaces/Driver Azimutal1/DIAG -> /Driver Azimutal1/DIAG
- U2 pad 12: /Interfaces/Driver Azimutal1/Index -> /Driver Azimutal1/Index
- U2 pad 14: /Interfaces/Driver Azimutal1/UART_RX -> /Driver Azimutal1/UART_RX
- U2 pad 16: /Interfaces/Driver Azimutal1/STEP -> /Driver Azimutal1/STEP
- U2 pad 17: unconnected-(U2-VREF-Pad17) -> /Driver Azimutal1/VREF
- U2 pad 19: /Interfaces/Driver Azimutal1/DIR -> /Driver Azimutal1/DIR
- U2 pad 2: /Interfaces/Driver Azimutal1/ENN -> /Driver Azimutal1/ENN
- U2 pad 20: /Interfaces/Driver Azimutal1/STDBY -> /Driver Azimutal1/STDBY
- U2 pad 21: /Interfaces/Driver Azimutal1/OA2 -> /Driver Azimutal1/OA2
- U2 pad 23: /Interfaces/Driver Azimutal1/BRB -> /Driver Azimutal1/BRB
- U2 pad 26: /Interfaces/Driver Azimutal1/OB1 -> /Driver Azimutal1/OB1
- U2 pad 27: /Interfaces/Driver Azimutal1/BRA -> /Driver Azimutal1/BRA
- U2 pad 7: /Interfaces/Driver Azimutal1/Spread -> /Driver Azimutal1/Spread
- U2 pad 8: unconnected-(U2-5VOUT-Pad8) -> Net-(U2-5VOUT)
- U2 pad 9: /Interfaces/Driver Azimutal1/MS1 -> /Driver Azimutal1/MS1
- U3 pad 1: /Interfaces/FB_3V3 -> /FB_3V3
- U5 pad 1: /Interfaces/FB_5V -> /FB_5V
Routing:
- net /Driver Azimutal1/STDBY: track 0.00 -> 11.6 mm, vias 0 -> 2
- net /Driver Azimutal1/Spread: track 0.00 -> 9.12 mm, vias 0 -> 2
- net Net-(U1-OUTPUT_RF): track 0.00 -> 6.73 mm
- net /Driver Azimutal1/UART_RX: track 0.00 -> 6.67 mm, vias 0 -> 2
- net /Driver Azimutal1/DIAG: track 0.00 -> 6.21 mm, vias 0 -> 2
- net Net-(U2-5VOUT): track 0.00 -> 5.26 mm
- net Net-(U3-SW): track 0.00 -> 3.59 mm
- net Net-(U2-VCP): track 0.00 -> 3.28 mm
- net Net-(U2-CPO): track 0.00 -> 2.91 mm
- net Net-(U2-CPI): track 0.00 -> 2.82 mm
- net Net-(LED2-+): track 0.00 -> 2.03 mm
- net GND: track 0.00 -> 1.74 mm
- net Net-(U3-CB): track 0.00 -> 1.71 mm
- net +20V: track 0.00 -> 1.10 mm
Other:
- board outline added: 53.5 x 78.3 mm
- copper layers 2 -> 4

Commit message: routage père quasi fini mais pb hiérarchique
Parts:
- removed C18: 33uF, EasyEDA:C1812
- added C1: C4532X7R1C336MT000N, EasyEDA:C1812, F.Cu at (152.2, 115.3)
- C13, C14, C17: value 33uF -> C4532X7R1C336MT000N
- TP1, TP2, TP3, TP4: footprint TestPoint:TestPoint_Pad_D2.5mm -> TestPoint:TestPoint_Pad_D1.5mm
- TP5: footprint TestPoint:TestPoint_Pad_D2.5mm -> TestPoint:TestPoint_Pad_1.5x1.5mm
- TP6, TP7: footprint TestPoint:TestPoint_Pad_2.5x2.5mm -> TestPoint:TestPoint_Pad_1.5x1.5mm
- moved C43 110.3 mm to (174.9, 118.4), turned to -90 degrees
- moved C46 109.6 mm to (179.1, 114.3), turned to 0 degrees
- moved C44 109.4 mm to (165.9, 105.5), turned to -90 degrees
- moved R21 107.2 mm to (184.1, 113.3)
- moved R8 105.0 mm to (166.4, 107.9)
- moved C38 104.3 mm to (179.7, 112.4), turned to 90 degrees
- moved C41 104.2 mm to (177.6, 118.4), turned to 90 degrees
- moved U7 103.7 mm to (175.9, 109.7), turned to 180 degrees
- moved R16 103.6 mm to (169.6, 107.8), turned to -90 degrees
- moved C35 103.3 mm to (169.4, 112.9), turned to 180 degrees
- moved C42 101.1 mm to (179.7, 106.7), turned to -90 degrees
- moved C37 96.9 mm to (172.9, 115.4), turned to -90 degrees
- moved C39 96.1 mm to (175.7, 114.8), turned to 180 degrees
- moved U6 95.3 mm to (171.4, 103.4), turned to -90 degrees
- moved R12 94.8 mm to (171.4, 115.4), turned to 90 degrees
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Connections:
- net /Driver Azimutal1/OA1 renamed /EL_OA1
- net /Driver Azimutal1/OA2 renamed /EL_OA2
- net /Driver Azimutal1/OB1 renamed /EL_OB1
- net /Driver Azimutal1/OB2 renamed /EL_OB2
- net /Driver Elevation/OA1 renamed /AZ_OA1
- net /Driver Elevation/OA2 renamed /AZ_OA2
- net /Driver Elevation/OB1 renamed /AZ_OB1
- net /Driver Elevation/OB2 renamed /AZ_OB2
- C14 pad 2: +3V3 -> +5V
Routing:
- net /Driver Elevation/MS2: track 0.00 -> 41.0 mm, vias 0 -> 1
- net /Driver Azimutal1/UART_TX: track 0.00 -> 37.4 mm, vias 0 -> 2
- net /Driver Azimutal1/DIR: track 0.00 -> 36.5 mm, vias 0 -> 1
- net +20V: track 1.10 -> 36.0 mm, vias 0 -> 26
- net /Driver Azimutal1/UART_RX: track 6.67 -> 39.0 mm
- net /Driver Azimutal1/STEP: track 0.00 -> 31.5 mm, vias 0 -> 3
- net /Driver Azimutal1/Index: track 0.00 -> 30.3 mm, vias 0 -> 1
- net /Driver Azimutal1/ENN: track 0.00 -> 28.7 mm, vias 0 -> 2
- net /EL_OA2: track 0.00 -> 26.4 mm, vias 0 -> 2
- net /EL_OB2: track 0.00 -> 23.5 mm, vias 0 -> 5
- net /Driver Elevation/Spread: track 0.00 -> 22.7 mm, vias 0 -> 2
- net /Driver Azimutal1/STDBY: track 11.6 -> 33.2 mm
- net /Driver Elevation/MS1: track 0.00 -> 19.8 mm, vias 0 -> 1
- net /Driver Azimutal1/DIAG: track 6.21 -> 25.9 mm
- net /Driver Azimutal1/MS2: track 0.00 -> 19.5 mm, vias 0 -> 2
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- added copper zone on In2.Cu, net +20V
- added copper zone on In2.Cu, net +3V3
- added copper zone on In2.Cu, net +5V
- added copper zone on B.Cu, net GND
- added copper zone on F.Cu, net GND
- added copper zone on In1.Cu, net GND
Other:
- board size 53.5 x 78.3 mm -> 52.9 x 80.1 mm

Commit message: pcb père quasi fini
Parts:
- removed C22: 22nF, EasyEDA:C0805
- added C18: CL10C220JB8NNNC, EasyEDA:C0603, F.Cu at (159.8, 103.5)
- added G***: LOGO, EasyEDA:Logo_astrolab, B.Cu at (182.4, 94.0)
- added LED5: Rouge, EasyEDA:LED-SMD_L1.6-W0.8-R-RD, F.Cu at (160.7, 71.1)
- added LED6: Rouge, EasyEDA:LED-SMD_L1.6-W0.8-R-RD, F.Cu at (161.9, 119.1)
- added R22: 1KΩ, EasyEDA:R0603, F.Cu at (158.1, 71.1)
- added R23: 680, EasyEDA:R0603, F.Cu at (158.8, 119.1)
- C21: value 22nF -> 22pF; footprint EasyEDA:C0805 -> EasyEDA:C0603
- H1, H2: moved to B.Cu
- moved C21 15.4 mm to (151.1, 90.6), turned to 90 degrees
- moved TP2 15.3 mm to (181.2, 116.8)
- moved TP1 15.3 mm to (176.5, 102.2)
- moved C36 14.4 mm to (168.7, 116.1), turned to 180 degrees
- moved U6 11.6 mm to (172.0, 115.0), turned to 90 degrees
- moved C45 10.8 mm to (179.3, 115.6), turned to 90 degrees
- moved C39 10.1 mm to (175.5, 104.6), turned to 0 degrees
- moved C37 9.38 mm to (173.6, 106.0), turned to 180 degrees
- moved C44 9.36 mm to (172.2, 112.4), turned to 0 degrees
- moved C46 9.19 mm to (178.2, 105.2), turned to 90 degrees
- moved R21 7.21 mm to (184.1, 106.0)
- moved R20 7.11 mm to (184.2, 113.2), turned to 180 degrees
- moved C35 6.21 mm to (168.9, 106.7)
- moved R12 3.65 mm to (170.6, 119.0)
- moved R16 3.63 mm to (168.8, 111.3), turned to 90 degrees
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Connections:
- C21 pad 1: /FB_3V3 -> /FB_5V
- C21 pad 2: +3V3 -> +5V
- C23 pad 2: /EL_OA2 -> /AZ_OA2
- C25 pad 2: /Driver Azimutal1/BRB -> /Driver Azimutal1/BRA
- C26 pad 2: /Driver Azimutal1/BRA -> /Driver Azimutal1/BRB
- C29 pad 2: /EL_OA1 -> /AZ_OA1
- C31 pad 1: /AZ_OB2 -> /EL_OB2
- C32 pad 2: /AZ_OA1 -> /EL_OA1
- C33 pad 1: /AZ_OB1 -> /EL_OB1
- C34 pad 2: /AZ_OA2 -> /EL_OA2
- C5 pad 1: /EL_OB2 -> /AZ_OB2
- C6 pad 1: /EL_OB1 -> /AZ_OB1
- CN3 pad 1: /EL_OA1 -> /AZ_OA1
- CN3 pad 2: /EL_OA2 -> /AZ_OA2
- CN3 pad 3: /EL_OB1 -> /AZ_OB1
- CN3 pad 4: /EL_OB2 -> /AZ_OB2
- CN4 pad 1: /AZ_OA1 -> /EL_OA1
- CN4 pad 2: /AZ_OA2 -> /EL_OA2
- CN4 pad 3: /AZ_OB1 -> /EL_OB1
- CN4 pad 4: /AZ_OB2 -> /EL_OB2
- H1 pad 3: +3V3 -> GND
- H1 pad 4: unconnected-(H1-Pad4) -> +3V3
- H1 pad 5: unconnected-(H1-Pad5) -> +3V3
- H1 pad 6: unconnected-(H1-Pad6) -> GND
- H1 pad 7: unconnected-(H1-Pad7) -> GND
- H1 pad 8: unconnected-(H1-Pad8) -> GND
- R1 pad 2: /Driver Azimutal1/BRA -> /Driver Azimutal1/BRB
- R2 pad 2: /Driver Azimutal1/BRB -> /Driver Azimutal1/BRA
- U2 pad 1: /EL_OB2 -> /AZ_OB2
- U2 pad 21: /EL_OA2 -> /AZ_OA2
- U2 pad 23: /Driver Azimutal1/BRB -> /Driver Azimutal1/BRA
- U2 pad 24: /EL_OA1 -> /AZ_OA1
- U2 pad 26: /EL_OB1 -> /AZ_OB1
- U2 pad 27: /Driver Azimutal1/BRA -> /Driver Azimutal1/BRB
- U7 pad 1: /AZ_OB2 -> /EL_OB2
- U7 pad 21: /AZ_OA2 -> /EL_OA2
- U7 pad 24: /AZ_OA1 -> /EL_OA1
- U7 pad 26: /AZ_OB1 -> /EL_OB1
Routing:
- net /STBY_Elevation: track 0.00 -> 70.7 mm, vias 0 -> 4
- net /Driver Elevation/UART_RX: track 0.00 -> 49.0 mm, vias 0 -> 3
- net /Driver Elevation/UART_TX: track 0.00 -> 47.7 mm, vias 0 -> 1
- net /Driver Elevation/Index: track 0.00 -> 45.0 mm, vias 0 -> 1
- net /Driver Elevation/DIAG: track 6.57 -> 43.9 mm
- net /Driver Elevation/ENN: track 0.00 -> 37.2 mm, vias 0 -> 1
- net /AZ_OA2: track 3.15 -> 26.9 mm, vias 0 -> 2
- net /AZ_OB2: track 3.22 -> 23.5 mm, vias 0 -> 5
- net /Driver Elevation/Spread: track 22.7 -> 38.9 mm, vias 2 -> 3
- net /AZ_OB1: track 3.12 -> 17.1 mm
- net /AZ_OA1: track 3.05 -> 16.7 mm, vias 0 -> 2
- net /Driver Elevation/MS2: track 41.0 -> 28.0 mm
- net +5V: track 13.9 -> 26.9 mm, vias 13 -> 12
- net /Driver Elevation/STEP: track 0.00 -> 12.9 mm, vias 0 -> 1
- net /Driver Elevation/BRA: track 0.00 -> 12.5 mm
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Other:
- board text added: "3.3V"
- board text added: "5V"
- board text added: "Azimuthal"
- board text added: "DIAG"
- board text added: "DIR"
- board text added: "ENN"
- board text added: "El_STDBY"
- board text added: "GND"
- board text added: "INDEX"
- board text added: "MS1"
- board text added: "MS2"
- board text added: "STDBY"
- board text added: "STEP"
- board text added: "Spread"
- board text added: "UART_RX"
- board text added: "UART_TX"
- board text added: "Élévation"
