File: Hardware/PCB/PCB_Pere/KiCad_Pere/PCB_Pere_V1/PCB_Pere_V1.kicad_sch (KiCad schematic)
At the start: 4 parts, among them CN1 B4B-PH-K-S, CN2 B4B-PH-K-S, U1 TMC2209-LA-T, U2 TMC2209-LA-T

Commit message: avancement schematic fils
Parts:
- removed CN1: B4B-PH-K-S, EasyEDA:CONN-TH_B4B-PH-K-S, symbol EasyEDA:B4B-PH-K-S
- removed U1, U2: TMC2209-LA-T, EasyEDA:QFN-28_L5.0-W5.0-P0.50-BL-EP, symbol EasyEDA:TMC2209-LA-T
- added H1: PZ254-1-20-Z-8.5, EasyEDA:HDR-TH_20P-P2.54-V-M, symbol EasyEDA:PZ254-1-20-Z-8.5
- added H2: PZ254-1-10-Z-8.5, EasyEDA:HDR-TH_10P-P2.54-V-M, symbol EasyEDA:PZ254-1-10-Z-8.5
- added U3, U4: LMR51625XDDCR_C44750835, EasyEDA:SOT-23-6_L2.9-W1.6-P0.95-LS2.9-BL, symbol EasyEDA:LMR51625XDDCR_C44750835
Connections:
- net Driver Azimutal/OA1: now reaches CN2.1
- net Driver Azimutal/OA2: now reaches CN2.2
- net Driver Azimutal/OB1: now reaches CN2.3
- net Driver Azimutal/OB2: now reaches CN2.4
Other:
- added sheet Driver Azimutal (Driver_azimutal.kicad_sch)
- moved on the sheet: CN2

Commit message: mise à jour PCB père
Parts:
- removed CN2: B4B-PH-K-S, EasyEDA:CONN-TH_B4B-PH-K-S, symbol EasyEDA:B4B-PH-K-S
- removed U4: LMR51625XDDCR_C44750835, EasyEDA:SOT-23-6_L2.9-W1.6-P0.95-LS2.9-BL, symbol EasyEDA:LMR51625XDDCR_C44750835
- added C13, C14, C17, C18: 33uF, EasyEDA:C1812, symbol EasyEDA:C4532X7R1C336M250KC
- added C15, C16, C19, C20: 100nF, EasyEDA:C0603, symbol EasyEDA:CC0603KRX7R9BB104
- added C21, C22: 22nF, EasyEDA:C0805, symbol EasyEDA:CL21B223KBANNNC
- added C7, C8: 2.2uF, EasyEDA:C1206, symbol EasyEDA:TCC1206X7R225K500FT
- added CN3: B4B-PH-K-S, EasyEDA:CONN-TH_B4B-PH-K-S, symbol EasyEDA:B4B-PH-K-S
- added L1: 10uH, EasyEDA:IND-SMD_L5.4-W5.2_FAUL0530-100MT, symbol EasyEDA:FAUL0530-100MT
- added L4: 15uF, EasyEDA:IND-SMD_L7.0-W6.6_MCW-0650-220, symbol EasyEDA:FAUL0630-150MT
- added R6: 53.6kR, EasyEDA:R0603, symbol EasyEDA:ARG03FTC5362
- added R7: 31.6kR, EasyEDA:R0603, symbol EasyEDA:ARG03FTC3162
- added R8, R9: 10.2kR, EasyEDA:R0603, symbol EasyEDA:ARG03FTC10R2
- added U5: Buck LMR51625, EasyEDA:SOT-23-6_L2.9-W1.6-P0.95-LS2.9-BL, symbol EasyEDA:LMR51625XDDCR_C44750835
- U3: value LMR51625XDDCR_C44750835 -> Buck LMR51625
Connections:
- net FB_3V3: now reaches U3.1 (FB)
- net FB_3V3: now also C21.1, R7.1, R9.2
- net +20V: now reaches U3.2 (EN)
- net +20V: now also U3.3 (VIN), C19.2, C20.2, C7.2, C8.2, U5.2 (EN), U5.3 (VIN)
- net GND: now reaches U3.4 (GND)
- net GND: now also C13.1, C14.1, C17.1, C18.1, C19.1, C20.1, C7.1, C8.1, R8.1, R9.1, U5.4 (GND)
- net at U3.5 (SW): now also C15.2, L1.1
- net at U3.6 (CB): now also C15.1
- new net: C16.2, L4.1, U5.5 (SW)
- new net: C16.1, U5.6 (CB)
- new net +3V3: C13.2, C14.2, C21.2, L1.2, R7.2
- new net +5V: C17.2, C18.2, C22.2, L4.2, R6.2
- new net Driver Azimutal1/OA1: CN3.1
- new net Driver Azimutal1/OA2: CN3.2
- new net Driver Azimutal1/OB1: CN3.3
- new net FB_5V: C22.1, R6.1, R8.2, U5.1 (FB)
Other:
- removed sheet Driver Azimutal
- added sheet Driver Azimutal1 (Driver_azimutal.kicad_sch)
- moved on the sheet: U3

Commit message: Routage toujours en attente oui je sais ça prend 10 000  ans mais it is what is
Parts:
- removed R6: 53.6kR, EasyEDA:R0603, symbol EasyEDA:ARG03FTC5362
- removed R7: 31.6kR, EasyEDA:R0603, symbol EasyEDA:ARG03FTC3162
- removed R8, R9: 10.2kR, EasyEDA:R0603, symbol EasyEDA:ARG03FTC10R2
- added C23, C29, C31, C32, C33, C34, C5, C6: 490pF, EasyEDA:C0603, symbol EasyEDA:0603B471K500NT
- added C27, C28: 330uF, EasyEDA:CAP-SMD_BD10.0-L10.3-W10.3-LS11.0-FD, symbol EasyEDA:RVT1H331M1010
- added C3: 2.2uF, EasyEDA:C1206, symbol EasyEDA:TCC1206X7R225K500FT
- added CN1: B2B-PH-K-S-GW, EasyEDA:CONN-TH_B2B-PH-K-S, symbol EasyEDA:B2B-PH-K-S-GW
- added CN4: B4B-PH-K-S, EasyEDA:CONN-TH_B4B-PH-K-S, symbol EasyEDA:B4B-PH-K-S
- added R11, R6: 47k, EasyEDA:R0603, symbol EasyEDA:0603WAF4702T5E
- added R13: 1KΩ, EasyEDA:R0603, symbol EasyEDA:0603WAF1001T5E
- added R7: 9.1k, EasyEDA:R0603, symbol EasyEDA:0603WAF9101T5E
- added R9: 15k, EasyEDA:R0603, symbol EasyEDA:0603WAF1502T5E
- added TP1, TP2, TP3, TP4, TP5: TestPoint, TestPoint:TestPoint_Pad_D2.5mm, symbol Connector:TestPoint
- added TP6, TP7: TestPoint, TestPoint:TestPoint_Pad_2.5x2.5mm, symbol Connector:TestPoint
Connections:
- net +20V: now also C27.1, C28.1, C3.2, CN1.1, TP7.1
- net +3V3: now also H1.3, R11.1, TP5.1
- net +5V: now also H1.2, R6.2, TP6.1
- net Driver Azimutal1/DIAG: now also H1.17
- net Driver Azimutal1/DIR: now also H1.14
- net Driver Azimutal1/ENN: now also H1.12
- net Driver Azimutal1/Index: now also H1.18
- net Driver Azimutal1/MS1: now also H1.15
- net Driver Azimutal1/MS2: now also H1.16
- net Driver Azimutal1/OA1: now also C29.2
- net Driver Azimutal1/OA2: now also C23.2
- net Driver Azimutal1/OB1: now also C6.1
- net Driver Azimutal1/OB2: now also CN3.4, C5.1
- net Driver Azimutal1/STEP: now also H1.11
- net Driver Azimutal1/Spread: now also H1.13
- net Driver Azimutal1/UART_RX: now also H1.20
- net Driver Azimutal1/UART_TX: now also H1.19
- net FB_3V3: now also R11.2, R9.2
- net FB_5V: now also R6.1, R7.2
- net GND: now also H1.1, C23.1, C27.2, C28.2, C29.1, C31.2, C32.1, C33.2, C34.1, C5.2, C6.2, CN1.2, R13.1, R7.1, R9.1
- net Driver Azimutal1/STDBY: now reaches H1.10
- net STBY_Elevation: now reaches H1.9
- net Driver Elevation/UART_TX: now reaches H2.1
- net Driver Elevation/STEP: now reaches H2.10
- net Driver Elevation/UART_RX: now reaches H2.2
- net Driver Elevation/Index: now reaches H2.3
- net Driver Elevation/DIAG: now reaches H2.4
- net Driver Elevation/MS2: now reaches H2.5
- net Driver Elevation/MS1: now reaches H2.6
- net Driver Elevation/DIR: now reaches H2.7
- net Driver Elevation/Spread: now reaches H2.8
- net Driver Elevation/ENN: now reaches H2.9
- new net: C3.1, R13.2
- new net Driver Azimutal1/BRA: TP3.1
- new net Driver Azimutal1/BRB: TP4.1
- new net Driver Elevation/BRA: TP1.1
- new net Driver Elevation/BRB: TP2.1
- new net Driver Elevation/OA1: C32.2, CN4.1
- new net Driver Elevation/OA2: C34.2, CN4.2
- new net Driver Elevation/OB1: C33.1, CN4.3
- new net Driver Elevation/OB2: C31.1, CN4.4
- no-connect marks 0 -> 5
Other:
- added sheet Driver Elevation (Driver_elevation.kicad_sch)
- sheet Driver Azimutal1 ports: added BRA, BRB, STDBY; removed none
- note added: "Alimentation 3.3V"
- note added: "Alimentation 5V"
- note added: "Driver Azimutal"
- note added: "Driver Elévation"
- note added: "Estimation de la tension en fonction des résistances de feedback : Vout = 0.8*(1+47k/15k) = 3.31V"
- note added: "Estimation de la tension en fonction des résistances de feedback : Vout = 0.8*(1+47k/9.1k) = 4.93V"
- note added: "Filtrage et stockage d'énergie"
- note added: "Penser à prévenir que STEP est connecté au TIM tandis que le GPIO nommé STEP servira pour le SPREAD"
- moved on the sheet: C13, C14, C15, C16, C17, C18, C19, C20, C21, C22, C7, C8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

Commit message: routage père quasi fini mais pb hiérarchique
Parts:
- removed C13, C14, C17, C18: 33uF, EasyEDA:C1812, symbol EasyEDA:C4532X7R1C336M250KC
- added C1, C13, C14, C17: C4532X7R1C336MT000N, EasyEDA:C1812, symbol EasyEDA:C4532X7R1C336MT000N
- TP1, TP2, TP3, TP4: footprint TestPoint:TestPoint_Pad_D2.5mm -> TestPoint:TestPoint_Pad_D1.5mm
- TP5: footprint TestPoint:TestPoint_Pad_D2.5mm -> TestPoint:TestPoint_Pad_1.5x1.5mm
- TP6, TP7: footprint TestPoint:TestPoint_Pad_2.5x2.5mm -> TestPoint:TestPoint_Pad_1.5x1.5mm
Connections:
- net +3V3: now also C1.2, C13.2
- net +5V: now also C14.2, C17.2
- net GND: now also C1.1, C13.1, C14.1, C17.1
- net Driver Azimutal1/OA1 renamed EL_OA1
- net Driver Azimutal1/OA2 renamed EL_OA2
- net Driver Azimutal1/OB1 renamed EL_OB1
- net Driver Azimutal1/OB2 renamed EL_OB2
- net Driver Elevation/OA1 renamed AZ_OA1
- net Driver Elevation/OA2 renamed AZ_OA2
- net Driver Elevation/OB1 renamed AZ_OB1
- net Driver Elevation/OB2 renamed AZ_OB2
Other:
- moved on the sheet: CN3, CN4

Commit message: pcb père quasi fini
Parts:
- removed C21, C22: 22nF, EasyEDA:C0805, symbol EasyEDA:CL21B223KBANNNC
- added C18: CL10C220JB8NNNC, EasyEDA:C0603, symbol EasyEDA:CL10C220JB8NNNC
- added C21: 22pF, EasyEDA:C0603, symbol EasyEDA:CL10C220JB8NNNC
- added LED5, LED6: Rouge, EasyEDA:LED-SMD_L1.6-W0.8-R-RD, symbol EasyEDA:KT-0603R
- added R22: 1KΩ, EasyEDA:R0603, symbol EasyEDA:0603WAF1001T5E
- added R23: 680, EasyEDA:R0603, symbol EasyEDA:0603WAF6800T5E
Connections:
- net +3V3: now also H1.4, H1.5, C18.2, R23.1; no longer H1.3
- net +5V: now also C21.2, R22.1
- net AZ_OA1: now also C29.2, CN3.1; no longer C32.2, CN4.1
- net AZ_OA2: now also C23.2, CN3.2; no longer C34.2, CN4.2
- net AZ_OB1: now also C6.1, CN3.3; no longer C33.1, CN4.3
- net AZ_OB2: now also C5.1, CN3.4; no longer C31.1, CN4.4
- net Driver Elevation/UART_RX: now also H2.1; no longer H2.2
- net Driver Elevation/UART_TX: now also H2.2; no longer H2.1
- net EL_OA1: now also C32.2, CN4.1; no longer C29.2, CN3.1
- net EL_OA2: now also C34.2, CN4.2; no longer C23.2, CN3.2
- net EL_OB1: now also C33.1, CN4.3; no longer C6.1, CN3.3
- net EL_OB2: now also C31.1, CN4.4; no longer C5.1, CN3.4
- net FB_3V3: now also C18.1
- net FB_5V: now also C21.1
- net GND: now also H1.3, H1.6, H1.7, H1.8, LED5.2 (K), LED6.2 (K)
- new net: LED6.1 (A), R23.2
- new net: LED5.1 (A), R22.2
- no-connect marks 5 -> 0
