File: Hardware/PCB/PCB_Pere/KiCad_Pere/PCB_Pere_V1/driver_azimutal.kicad_sch (KiCad schematic)
At the start: 0 parts

Commit message: MAJ Application
Parts:
- added C10, C12, C24, C25, C26, C30, C9: 100nF, EasyEDA:C0603, symbol EasyEDA:CC0603KRX7R9BB104
- added C11: 22nF, EasyEDA:C0805, symbol EasyEDA:CL21B223KBANNNC
- added C2, C4, C40: 2.2uF, EasyEDA:C1206, symbol EasyEDA:TCC1206X7R225K500FT
- added LED2: Yellow, EasyEDA:LED0805-R-RD, symbol EasyEDA:17-21SUYC_TR8
- added R1, R2: 120mΩ, EasyEDA:R2512, symbol EasyEDA:25121WF120LT4E
- added R10: 1KΩ, EasyEDA:R0603, symbol EasyEDA:0603WAF1001T5E
- added R14: TC33X-2-103E, EasyEDA:RES-ADJ-SMD_3P-L3.0-W3.8-P1.75-BR, symbol EasyEDA:TC33X-2-103E
- added R15: 10k, EasyEDA:R0603, symbol EasyEDA:0603WAF1002T5E
- added R3, R4: 100kΩ, EasyEDA:R0603, symbol EasyEDA:0603WAF1003T5E
- added R5: 1kΩ, EasyEDA:R0603, symbol EasyEDA:0603WAF1001T5E
- added U2: TMC2209-LA-T, EasyEDA:QFN-28_L5.0-W5.0-P0.50-BL-EP, symbol EasyEDA:TMC2209-LA-T
- added U4: 8132H-10.000NL33DTL, EasyEDA:OSC-SMD_4P-L3.2-W2.5-BL, symbol EasyEDA:8132H-10.000NL33DTL
Connections:
- new net: C9.1, U2.6 (VCP)
- new net: R14.3, R15.1
- new net: C2.1, R15.2, U2.8 (5VOUT)
- new net: LED2.1 (+), R5.1
- new net: U2.13 (CLK), U4.3 (OUTPUT_RF)
- new net: C11.2, U2.4 (CPO)
- new net: C11.1, U2.5 (CPI)
- new net +20V: C10.2, C12.2, C4.2, C40.2, C9.2, U2.22 (VS), U2.28 (VS)
- new net +3V3: C24.2, C30.1, U2.15 (VCC_IO), U4.4 (VCC)
- new net BRA: C25.2, R2.2, U2.23 (BRA)
- new net BRB: C26.2, R1.2, U2.27 (BRB)
- new net DIAG: R5.2, U2.11 (DIAG)
- new net DIR: U2.19 (DIR)
- new net ENN: U2.2 (ENN)
- new net GND: C10.1, C12.1, C2.2, C24.1, C25.1, C26.1, C30.2, C4.1, C40.1, LED2.2 (-), R1.1, R14.1, R2.1, R3.1, R4.1, U2.18 (GND), U2.29 (EP), U2.3 (GND), U4.2 (GND)
- new net Index: U2.12 (INDEX)
- new net MS1: U2.9 (MS1_AD0)
- new net MS2: U2.10 (MS2_AD1)
- new net OA1: U2.24 (OA1)
- new net OA2: U2.21 (OA2)
- new net OB1: U2.26 (OB1)
- new net OB2: U2.1 (OB2)
- new net STDBY: R3.2, U2.20 (STDBY)
- new net STEP: U2.16 (STEP)
- new net Spread: R4.2, U2.7 (SPREAD)
- new net UART_RX: R10.2, U2.14 (PDN_UART)
- new net UART_TX: R10.1
- new net VREF: R14.2, U2.17 (VREF)
- no-connect marks 0 -> 2
Other:
- note added: "Driver Elévation"
- note added: "Le Vref est réglable entre 0 et 2.5V pour pouvoir limiter le courant en mode autonome. 0Ohms -> 0V 10kOhms -> 2.5V : Ampérage maximal : 1.64A RMS (moteur 1.7A) Le réglage du potentiomètre n'est pas nécessaire avec l'utilisation de l'UART mais il reste possible d'utiliser Vref dans les paramètres de l'UART"
- note added: "Reste à faire : ajouter des condensateurs en entrée de puissance voir si on a besoin du standby + ajouter pulldown keskeusé keut le 5Vout ? Voir comment gérer les sense resistor avec Vref et les BRB"
