File: Hardware/PCB/PCB_Fils/PCB_Fils.kicad_pcb (KiCad board)
At the start: 4 copper layers, 30.8 x 30.5 mm, 31 parts, among them U1 S6B-PH-K-S-, U2 MCP23008-E/ML, U3 TPS22918DBVR, U4 BNO055, U5 TPS22918DBVR, U6 B8B-PH-K-S_FILS, X2 X701532768KGD4GI

Commit message: last version + Ajout du PCB Fils FINI?
Other:
- board text added: "Carte Fils"
- board text added: "L'Index Stellaire L'ASTROLAB"
