File: Hardware/PCB/PCB_Pere/KiCad_Pere/PCB_Pere_V1/_restore_backup_2026-10-16T18-20-06-566/driver_azimutal.kicad_sch (KiCad schematic)
At the start: 0 parts

Commit message: MAJ Application
Parts:
- added C1, C2: 330uF, EasyEDA:CAP-SMD_BD10.0-L10.3-W10.3-LS11.0-FD, symbol EasyEDA:RVT1H331M1010
- added C3, C4, C6: 100nF, EasyEDA:C0603, symbol EasyEDA:CC0603KRX7R9BB104
- added C5: 22nF, EasyEDA:C0805, symbol EasyEDA:CL21B223KBANNNC
- added LED1: Yellow, EasyEDA:LED0805-R-RD, symbol EasyEDA:17-21SUYC_TR8
- added R1, R2: 1KΩ, EasyEDA:R0603, symbol EasyEDA:0603WAF1001T5E
- added R3: 100kΩ, EasyEDA:R0603, symbol EasyEDA:0603WAF1003T5E
- added U1: TMC2209-LA-T, EasyEDA:QFN-28_L5.0-W5.0-P0.50-BL-EP, symbol EasyEDA:TMC2209-LA-T
- added X2: 12 MHz, EasyEDA:CRYSTAL-SMD_4P-L3.2-W2.5-BL, symbol EasyEDA:X322512MSB4SI
Connections:
- new net: C1.1, C2.1, C3.2, C4.2, U1.22 (VS), U1.28 (VS)
- new net: C4.1, U1.6 (VCP)
- new net: LED1.1 (+), R2.1
- new net: U1.13 (CLK), X2.3 (OSC2)
- new net: C5.2, U1.4 (CPO)
- new net: C5.1, U1.5 (CPI)
- new net +3V3: C6.2, U1.15 (VCC_IO)
- new net DIAG: R2.2, U1.11 (DIAG)
- new net DIR: U1.19 (DIR)
- new net ENN: U1.2 (ENN)
- new net GND: C1.2, C2.2, C3.1, C6.1, LED1.2 (-), R3.1, U1.18 (GND), U1.29 (EP), U1.3 (GND), X2.2 (GND), X2.4 (GND)
- new net Index: U1.12 (INDEX)
- new net MS1: U1.9 (MS1_AD0)
- new net MS2: U1.10 (MS2_AD1)
- new net OA1: U1.24 (OA1)
- new net OA2: U1.21 (OA2)
- new net OB1: U1.26 (OB1)
- new net OB2: U1.1 (OB2)
- new net STDBY: U1.20 (STDBY)
- new net STEP: U1.16 (STEP)
- new net Spread: R3.2, U1.7 (SPREAD)
- new net UART_RX: R1.2, U1.14 (PDN_UART)
- new net UART_TX: R1.1
- no-connect marks 0 -> 1
Other:
- note added: "Led jaune de debug en plus d'un signal envoyé à la stm"
- note added: "Reste à faire : ajouter des condensateurs en entrée de puissance voir si on a besoin du standby + ajouter pulldown keskeusé keut le 5Vout ? Voir comment gérer les sense resistor avec Vref et les BRB"
- note added: "prende passe inductance pour les résistances de Rsa et RSB 0.5W, 1206"
